File: PCB/projects/1st Layer 2018v1/1stLayer2018v1.sch (EAGLE design)
At the start: 36 parts, among them U1 TEMT6000

Commit message: 0.1% progress
Parts:
- added C4: 0.1uF, rcl:C-EUC0603
- added U$3: 100k, JH:MCP41XXX
- R5: value 10K -> 10k; device SparkFun:RESISTOR0402-RES -> SparkFun-Resistors:RESISTOR0402
- U1: value TEMT6000 -> LIGHT_SENSORTEMT6000; device SparkFun:TEMT6000 -> SparkFun-Sensors:LIGHT_SENSORTEMT6000
Connections:
- new net N$10: U$3.PA0, U$3.PW0
- new net N$9: C4.1, U$3.VCC
- net 3.3V: now also C4.2, U$3.GND
Changed lines of the file:
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@@
 <drawing>
 <settings>
-<setting alwaysvectorfont="yes"/>
+<setting alwaysvectorfont="no"/>
 <setting verticaltext="up"/>
 </settings>
@@
 <part name="SUPPLY4" library="SparkFun-PowerSymbols" library_urn="urn:adsk.eagle:library:530" deviceset="3.3V" device=""/>
 <part name="CIN4" library="rcl" library_urn="urn:adsk.eagle:library:334" deviceset="C-EU" device="C1210" package3d_urn="urn:adsk.eagle:package:23619/2" value="22.0uF"/>
-<part name="R5" library="SparkFun" deviceset="RESISTOR" device="0402-RES" value="10K"/>
-<part name="U1" library="SparkFun" deviceset="TEMT6000" device=""/>
+<part name="R5" library="SparkFun-Resistors" library_urn="urn:adsk.eagle:library:532" deviceset="RESISTOR" device="0402" package3d_urn="urn:adsk.eagle:package:39657/1" value="10k"/>
+<part name="U1" library="SparkFun-Sensors" deviceset="LIGHT_SENSOR" device="TEMT6000"/>
 <part name="P+1" library="SparkFun-PowerSymbols" library_urn="urn:adsk.eagle:library:530" deviceset="3.3V" device=""/>
 <part name="FRAME2" library="SparkFun-Aesthetics" library_urn="urn:adsk.eagle:library:507" deviceset="FRAME-LETTER" device="" package3d_urn="urn:adsk.eagle:package:37121/1"/>
@@
 <part name="FRAME8" library="SparkFun-Aesthetics" library_urn="urn:adsk.eagle:library:507" deviceset="FRAME-LETTER" device="" package3d_urn="urn:adsk.eagle:package:37121/1"/>
 <part name="FRAME9" library="SparkFun-Aesthetics" library_urn="urn:adsk.eagle:library:507" deviceset="FRAME-LETTER" device="" package3d_urn="urn:adsk.eagle:package:37121/1"/>
-<part name="TPS5450_1" library="JH" library_urn="urn:adsk.eagle:library:6027132" deviceset="TPS5450" device="" package3d_urn="urn:adsk.eagle:package:6740528/2" value="5.1v"/>
-<part name="TPS5450_2" library="JH" library_urn="urn:adsk.eagle:library:6027132" deviceset="TPS5450" device="" package3d_urn="urn:adsk.eagle:package:6740528/2" value="3.1v"/>
+<part name="TPS5450_1" library="JH" library_urn="urn:adsk.eagle:library:6027132" deviceset="TPS5450" device="" package3d_urn="urn:adsk.eagle:package:6740528/3" value="5.1v"/>
+<part name="TPS5450_2" library="JH" library_urn="urn:adsk.eagle:library:6027132" deviceset="TPS5450" device="" package3d_urn="urn:adsk.eagle:package:6740528/3" value="3.1v"/>
 <part name="MAX1522" library="JH" library_urn="urn:adsk.eagle:library:6027132" deviceset="MAX1522EUT+T" device="" package3d_urn="urn:adsk.eagle:package:6740527/2" value="65v"/>
 <part name="P+3" library="SparkFun-PowerSymbols" library_urn="urn:adsk.eagle:library:530" deviceset="3.3V" device=""/>
@@
 <part name="R7" library="rcl" library_urn="urn:adsk.eagle:library:334" deviceset="R-EU_" device="R0603" package3d_urn="urn:adsk.eagle:package:23555/2" value="30k"/>
 <part name="R8" library="rcl" library_urn="urn:adsk.eagle:library:334" deviceset="R-EU_" device="R0603" package3d_urn="urn:adsk.eagle:package:23555/2" value="30k"/>
+<part name="U$3" library="JH" library_urn="urn:adsk.eagle:library:6027132" deviceset="MCP41XXX" device="" package3d_urn="urn:adsk.eagle:package:6868027/1" value="100k"/>
+<part name="C4" library="rcl" library_urn="urn:adsk.eagle:library:334" deviceset="C-EU" device="C0603" package3d_urn="urn:adsk.eagle:package:23616/2" value="0.1uF"/>
+<part name="GND8" library="SparkFun-PowerSymbols" library_urn="urn:adsk.eagle:library:530" deviceset="GND2" device="" value="GND"/>
+<part name="GND9" library="SparkFun-PowerSymbols" library_urn="urn:adsk.eagle:library:530" deviceset="GND2" device="" value="GND"/>
 </parts>
 <sheets>
@@
 <attribute name="VALUE" x="148.082" y="69.85" size="1.778" layer="96" rot="R90"/>
 </instance>
+<instance part="U$3" gate="G$1" x="91.44" y="43.18" smashed="yes">
+<attribute name="NAME" x="91.44" y="49.53" size="1.27" layer="95" font="vector" ratio="10" align="center"/>
+<attribute name="VALUE" x="91.44" y="34.29" size="1.143" layer="96" font="vector" ratio="10" align="center"/>
+</instance>
+<instance part="C4" gate="G$1" x="109.22" y="45.72" smashed="yes" rot="R90">
+<attribute name="NAME" x="108.839" y="47.244" size="1.778" layer="95" rot="R90"/>
+<attribute name="VALUE" x="113.919" y="47.244" size="1.778" layer="96" rot="R90"/>
+</instance>
+<instance part="GND8" gate="G$1" x="119.38" y="45.72" smashed="yes" rot="R90">
+<attribute name="VALUE" x="121.158" y="45.72" size="1.778" layer="96" rot="R90" align="top-center"/>
+</instance>
+<instance part="GND9" gate="G$1" x="76.2" y="38.1" smashed="yes" rot="R270">
+<attribute name="VALUE" x="74.422" y="38.1" size="1.778" layer="96" rot="R270" align="top-center"/>
+</instance>
 </instances>
 <busses>
@@
 <wire x1="81.28" y1="88.9" x2="81.28" y2="86.36" width="0.1524" layer="91"/>
 </segment>
+<segment>
+<pinref part="C4" gate="G$1" pin="2"/>
+<pinref part="GND8" gate="G$1" pin="3.3V"/>
+<wire x1="116.84" y1="45.72" x2="114.3" y2="45.72" width="0.1524" layer="91"/>
+</segment>
+<segment>
+<pinref part="GND9" gate="G$1" pin="3.3V"/>
+<pinref part="U$3" gate="G$1" pin="GND"/>
+<wire x1="78.74" y1="38.1" x2="81.28" y2="38.1" width="0.1524" layer="91"/>
+</segment>
 </net>
 <net name="N$7" class="0">
@@
 </segment>
 </net>
+<net name="N$9" class="0">
+<segment>
+<pinref part="U$3" gate="G$1" pin="VCC"/>
+<pinref part="C4" gate="G$1" pin="1"/>
+<wire x1="101.6" y1="45.72" x2="106.68" y2="45.72" width="0.1524" layer="91"/>
+</segment>
+</net>
+<net name="N$10" class="0">
+<segment>
+<pinref part="U$3" gate="G$1" pin="PW0"/>
+<wire x1="101.6" y1="40.64" x2="104.14" y2="40.64" width="0.1524" layer="91"/>
+<wire x1="104.14" y1="40.64" x2="104.14" y2="38.1" width="0.1524" layer="91"/>
+<pinref part="U$3" gate="G$1" pin="PA0"/>
+<wire x1="104.14" y1="38.1" x2="101.6" y2="38.1" width="0.1524" layer="91"/>
+</segment>
+</net>

Commit message: update
Parts:
- removed FRAME1, FRAME2, FRAME3, FRAME4, FRAME5, FRAME6, FRAME7, FRAME8, FRAME9: FRAME-LETTER, SparkFun-Aesthetics:FRAME-LETTER
- added D3: (no value), diode:SCHOTTKY-DIODESMD
- added Q1: 68V/98A/9.8mΩ, SparkFun-DiscreteSemi:MOSFET-NCH-FQP30N06L
Connections:
- new net GND: C3.2, C4.2, MAX1522.GND, U$3.GND, U$3.PB0
- new net N$11: D3.A, Q1.D
- new net N$12: D3.C, R6.2
- net 3.3V: now also C4.1, Q1.S, U$3.VCC; no longer C3.2, C4.2, MAX1522.GND, U$3.GND
- net N$10: now also R8.1
- net N$8: now also MAX1522.FB
- net N$9: now also MAX1522.EXT, Q1.G; no longer C4.1, U$3.VCC
Other:
- moved on the sheet: C1, C2, C3, C4, CBOOT1, CBOOT2, CIN1, CIN2, CIN3, CIN4, D1, D2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

Commit message: left new pill and adxl, cleaned up some symbols and wrong net names, have to make breakout pins for data pins
Parts:
- added 100YXJ: 100v/100uf, rcl:CPOL-USE5-10.5
- added C10: 1500pF, rcl:C-EUC0603
- added C5, C6: 1000uf, JH:100UF-CAP
- added C7: 0.1uF, rcl:C-EUC0603
- added C8: 33nF, rcl:C-EUC0603
- added C9: 680uF/16V, rcl:CPOL-USE3.5-8
- added CIN5: 22.0uF, rcl:C-EUC1210
- added Q2: 5.8A/30V/35mΩ, SparkFun-DiscreteSemi:MOSFET-NCH-AO3404A
- added Q3: 60V/32A/35mΩ, SparkFun-DiscreteSemi:MOSFET-NCH-FQP30N06L
- added R10, R12, R19: 4.7k, rcl:R-EU_R0603
- added R11, R13, R14, R16, R23, R9: 1k, rcl:R-EU_R0603
- added R15: 100k, rcl:R-EU_R0603
- added R17, R20, R21, R22: 10k, rcl:R-EU_R0603
- added R18: 1.5k, rcl:R-EU_R0603
- added R24: 20, rcl:R-EU_R0603
- added SS54, SS54-1, SS54-2: 5A/40V, diode:SCHOTTKY-DIODESMD
- added STP75NF75: 75V/80A/11mΩ, SparkFun-DiscreteSemi:MOSFET-NCH-FQP30N06L
- added U$4, U$5: (no value), JH:CDRH127
- added U$6: VNH5050A, JH:VNH5050A
- added U2: CD74HC4067SM96, SparkFun-IC-Logic:74HC4067SM96
- D1: value (none) -> 1N4728; device diode:SCHOTTKY-DIODESMD -> diode:1N4728
- D2: value (none) -> 1N5401; device diode:SCHOTTKY-DIODESMD -> diode:1N5400
- Q1: value 68V/98A/9.8mΩ -> 35A/25V/8.5mΩ; device SparkFun-DiscreteSemi:MOSFET-NCH-FQP30N06L -> SparkFun-DiscreteSemi:MOSFET-NCH-FDD8780
- R5: device SparkFun-Resistors:RESISTOR0402 -> SparkFun-Resistors:10KOHM-0603-1/10W-1%
- SS510: value (none) -> 5A/100V
- renumbered D3 to SS510
Connections:
- new net 60V: 100YXJ.+, C5.+, C6.+, R6.2, SS510.C
- new net CS: R16.2
- new net EN_A: R9.2
- new net EN_B: R11.1
- new net IN_A: R14.2
- new net IN_B: R13.1
- new net N$13: R14.1, U$6.IN_A
- new net N$14: R11.2, R12.2, U$6.EN_B
- new net N$15: R13.2, U$6.IN_B
- new net N$16: R17.2, R19.1, U$6.PWM_IN
- new net N$17: R16.1, R18.1, U$6.CS
- new net N$18: Q2.G, R21.2
- new net N$19: Q1.S, SS54.A, U$6.GND_A, U$6.GND_B
- new net N$20: Q1.G, R15.2, SS54.C
- new net N$21: R20.1, U$6.CS_DIS
- new net N$22: C10.2, Q2.D, Q3.S, R22.1
- new net N$23: Q3.G, R23.2
- new net N$24: D1.C, D2.C
- new net N$26: C10.1, R24.1
- new net OUT_A: U$6.OUT_A
- new net OUT_B: U$6.OUT_B
- new net PWM: C8.1, R17.1
- new net SOLENOID+: D1.A
- new net SOLENOID-: D2.A, Q3.D, R24.2
- net 12V: now also C9.+, CIN5.1, R15.1, R22.2, R23.1, U$4.1, U$5.1, U$6.VCC
- net 3.3V: now also C2.+, C7.1, R10.1, R12.1, R3.2, U2.EN, U2.VCC, XAL6060.2; no longer C1.-, C2.-, C3.1, CIN1.2, CIN2.2, CIN3.2, CIN4.2, D1.A, D2.A, MAX1522.!SHDN, MAX1522.SET, MAX1522.VCC, Q1.S, R2.1, R4.1, R5.1, TPS5450_1.GND, TPS5450_2.GND, U$1.C, U$2.C
- net 5V: now also C3.1, MAX1522.!SHDN, MAX1522.SET, MAX1522.VCC; no longer C2.+, R3.2, XAL6060.2
- net GND: now also 100YXJ.-, C1.-, C2.-, C5.-, C6.-, C7.2, C8.2, C9.-, CIN1.2, CIN2.2, CIN3.2, CIN4.2, CIN5.2, Q1.D, Q2.S, R18.2, R19.2, R2.1, R20.2, R21.1, R4.1, R5.1, SS54-1.A, SS54-2.A, STP75NF75.S, TPS5450_1.GND, TPS5450_2.GND, U$1.C, U$2.C, U2.GND
- net N$1: now also SS54-1.C; no longer D1.C
- net N$11: now also STP75NF75.D, U$4.2, U$5.2; no longer Q1.D
- net N$12: now also R10.2, R9.1, U$6.EN_A; no longer R6.2, SS510.C
- net N$5: now also SS54-2.C; no longer D2.C
- net N$9: now also STP75NF75.G; no longer Q1.G
