File: PCB/projects/TestV2/TestV2.sch (EAGLE design)
At the start: 109 parts, among them Q1 35A/25V/8.5mΩ, Q2 5.8A/30V/35mΩ, Q3 60V/32A/35mΩ, X1 USB-MINIB

Commit message: 8/12 PCB well well well so drunk the original commit name was 9/12 renamed all parts in schematic, then everything went downhill welp was in 1mm grid instead of 1.27mm forgot to check drc before routing and placing everything, will redo all the placements soon lesson: dont be stupid thanks the upside is we may actually have a very legit motor driver and new pill module rip
Parts:
- removed C11, C12: 47pF, rcl:C-EUC0603
- removed C14, C15, C16, C17: 1uF, rcl:C-EUC0603
- removed C18: 22uf, rcl:C-EUC1210
- removed C19, C20: 18pF, rcl:C-EUC0603
- removed C21: 22uF, rcl:C-EUC1210
- removed C8: 33nF, rcl:C-EUC0603
- removed C9: 680uF/16V, rcl:CPOL-USE3.5-8
- removed D2: 1N5401, diode:1N5400
- removed D3: RED, SparkFun-LED:LED-RED1206
- removed D4: SS14, diode:DIODE-DO-214AC
- removed OSC: 8MHz, SparkFun-Clocks:CRYSTALSMD-HC49UP
- removed Q1: 35A/25V/8.5mΩ, SparkFun-DiscreteSemi:MOSFET-NCH-FDD8780
- removed R10, R12, R19: 4.7k, rcl:R-EU_R0603
- removed R11, R13, R14, R16, R25, R36, R9: 1k, rcl:R-EU_R0603
- removed R15: 100k, rcl:R-EU_R0603
- removed R17, R20, R34, R35: 10k, rcl:R-EU_R0603
- removed R18, R28: 1.5k, rcl:R-EU_R0603
- removed R26, R27, R31: 22, rcl:R-EU_R0603
- removed R29: 300ohm bead, rcl:R-EU_R0402
- removed RESET: TAC_SWITCHSMD, SparkFun-Retired:TAC_SWITCHSMD
- removed SS54: 5A/40V, diode:SCHOTTKY-DIODESMD
- added 1C1, 1C2, 1C3, 1C4, 5C10, 5C5, 5C7, 5C8, 5C9: 1uF, rcl:C-EUC0603
- added 3UP-R1, 3UP-R2, 5R1, 5R5, 6R1, 6R2, 6R3, 6R4, 6R5: 1k, rcl:R-EU_R0603
- added 4D2: 1N5401, diode:1N5400
- added 5C1, 5C2: 18pF, rcl:C-EUC0603
- added 5C3, 5C4: 47pF, rcl:C-EUC0603
- added 5C6: 1uf, rcl:C-EUC0603
- added 5D1: SS14, diode:DIODE-DO-214AC
- added 5DOWN-R1, 5R3, 5R4: 22, rcl:R-EU_R0603
- added 5F1: 300ohm bead, rcl:R-EU_R0402
- added 5LED1: RED, SparkFun-LED:LED-RED1206
- added 5OSC: 8MHz, SparkFun-Clocks:CRYSTALSMD-HC49UP
- added 5R2, 5R6, 6DOWN-R3, 6R6: 10k, rcl:R-EU_R0603
- added 5RESET: TAC_SWITCHSMD, SparkFun-Retired:TAC_SWITCHSMD
- added 5UP-R1, 6DOWN-R1: 1.5k, rcl:R-EU_R0603
- added 6C1: 33nF, rcl:C-EUC0603
- added 6COUT: 680uF/16V, rcl:CPOL-USE3.5-8
- added 6D1: 5A/40V, diode:SCHOTTKY-DIODESMD
- added 6DOWN-R2, 6UP-R1, 6UP-R2: 4.7k, rcl:R-EU_R0603
- added 6MOS1: AP86T02GH, SparkFun-DiscreteSemi:MOSFET-NCH-FDD8780
- added 6R7: 100k, rcl:R-EU_R0603
- 4MOS1: value 5.8A/30V/35mΩ -> AO3400
- 4MOS2: value 60V/32A/35mΩ -> STP75NF75
- VREGJUMPER: device SparkFun-Connectors:CONN_04LOCK -> SparkFun-Connectors:CONN_02LOCK
- renumbered 1LED3 to 1LED5, 2SDIO1 to 2D1, 2SDIO2 to 2D2, 3DIO1 to 3D1, C10 to 4CSNUB, D1 to 4D1, Q2 to 4MOS1, Q3 to 4MOS2, R21 to 4DOWN-R1, R22 to 4DOWN-R2, R23 to 4R1, R24 to 4RSNUB
Connections:
- removed net 33: R25.2, UC1.PB1/ADC12_IN9/TIM3_CH4
- removed net N$41: U$7.OUT, VREGJUMPER.3
- removed net OUT_A: MOTOROUT.1, U$6.OUT_A
- removed net OUT_B: MOTOROUT.3, U$6.OUT_B
- new net N$25: 3UP-R1.1, MAX1522.!SHDN
- new net N$29: 3UP-R2.1, MAX1522.SET
- new net N$31: 5R5.2, UC1.PB1/ADC12_IN9/TIM3_CH4
- new net N$32: MOTOROUT.3, U$6.OUT_A
- new net N$33: MOTOROUT.1, U$6.OUT_B
- net 0: now also STM32OUT1.20; no longer STM32OUT1.19
- net 1: now also STM32OUT1.19; no longer STM32OUT1.18
- net 12V: now also 6COUT.+, 6R7.1; no longer C9.+, R15.1
- net 2: now also STM32OUT1.18; no longer STM32OUT1.17
- net 23_USBDP: now also 5C4.2, 5R4.1, 5UP-R1.1; no longer C12.2, R27.1, R28.1
- net 24_USBDM: now also 5C3.2, 5R3.1; no longer C11.2, R26.1
- net 3.3V: now also 1C1.1, 1C2.1, 1C3.1, 1C4.1, 5C10.1, 5C6.1, 5C7.1, 5C8.1, 5C9.1, 5R2.2, 5UP-R1.2, 6UP-R1.1, 6UP-R2.1, U$7.OUT; no longer C14.1, C15.1, C16.1, C17.1, C18.1, R10.1, R12.1, R28.2, R35.2, VREGJUMPER.4
- net 32: now also 5R6.1; no longer R34.1
- net 5V: now also 3UP-R1.2, 3UP-R2.2, 5C5.1, 5D1.C; no longer C21.1, D4.C, MAX1522.!SHDN, MAX1522.SET
- net AGND: now also 5C10.2, 5F1.1, STM32OUT1.7; no longer C14.2, R29.1
- net CS: now also 6R5.2; no longer R16.2
- net EN_A: now also 6R1.2; no longer R9.2
- net EN_B: now also 6R2.1; no longer R11.1
- net GND: now also 1C1.2, 1C2.2, 1C3.2, 1C4.2, 5C1.2, 5C2.2, 5C3.1, 5C4.1, 5C5.2, 5C6.2, 5C7.2, 5C8.2, 5C9.2, 5DOWN-R1.1, 5F1.2, 5LED1.C, 5R1.1, 6C1.2, 6COUT.-, 6DOWN-R1.2, 6DOWN-R2.2, 6DOWN-R3.2, 6MOS1.D; no longer C11.1, C12.1, C15.2, C16.2, C17.2, C18.2, C19.2, C20.2, C21.2, C8.2, C9.-, D3.C, Q1.D, R18.2, R19.2, R20.2, R29.2, R31.1, R36.1
- net IN_A: now also 6R3.2; no longer R14.2
- net IN_B: now also 6R4.1; no longer R13.1
- net N$12: now also 6R1.1, 6UP-R2.2; no longer R10.2, R9.1
- net N$13: now also 6R3.1; no longer R14.1
- net N$14: now also 6R2.2, 6UP-R1.2; no longer R11.2, R12.2
- net N$15: now also 6R4.2; no longer R13.2
- net N$16: now also 6DOWN-R2.1, 6R6.2; no longer R17.2, R19.1
- net N$17: now also 6DOWN-R1.1, 6R5.1; no longer R16.1, R18.1
- net N$19: now also 6D1.A, 6MOS1.S; no longer Q1.S, SS54.A
- net N$20: now also 6D1.C, 6MOS1.G, 6R7.2; no longer Q1.G, R15.2, SS54.C
- net N$21: now also 6DOWN-R3.1; no longer R20.1
- net N$24: now also 4D2.C; no longer D2.C
- net N$27: now also 5R1.2, 5RESET.1, 5RESET.2; no longer R36.2, RESET.1, RESET.2
- net N$28: now also 5LED1.A, 5R5.1; no longer D3.A, R25.1
- net N$30: now also 5R6.2; no longer R34.2
- net N$36: now also 5DOWN-R1.2; no longer R31.2
- net N$59: now also 5R3.2; no longer R26.2
- net N$60: now also 5R4.2; no longer R27.2
- net OSC_IN: now also 5C2.1, 5OSC.2; no longer C19.1, OSC.2
- net OSC_OUT: now also 5C1.1, 5OSC.1; no longer C20.1, OSC.1
- net PWM: now also 6C1.1, 6R6.1; no longer C8.1, R17.1
- net RESET: now also 5R2.1, 5RESET.3, 5RESET.4; no longer R35.1, RESET.3, RESET.4, STM32OUT1.7
- net SOLENOID-: now also 4D2.A, SOLENOIDOUT.1; no longer D2.A, SOLENOIDOUT.3
- net SOLENOIDON: no longer STM32OUT1.20
- net VCC_1: now also SOLENOIDOUT.3; no longer SOLENOIDOUT.1
- net V_USB: now also 5D1.A; no longer D4.A

Commit message: 11/12 PCB Updated own DRU file Updated even more stuff in schematic but quite minor, mostly flipping the 5mm screw terminal connections redid the pcb kinda redid the layout and managed to frkin manual route the stm32 new pill with 10mil traces oyas feelsgood super behind time again but lifes good
Parts:
- added 7C1, 7C3: 47uF, rcl:C-EUC0603
- added 7C2, 7C4: 1uF, rcl:C-EUC0603
- added 7R1, 7R3: (no value), rcl:R-EU_R0603
- added 7R2, 7R4: 100k, rcl:R-EU_R0603
- added 7UP-R1, 7UP-R2: 10k, rcl:R-EU_R0603
- added IR/OUT: (no value), SparkFun-Connectors:CONN_04LOCK
- added U1, U2: 38kHz, SparkFun-Sensors:TSOP38238
- added VSELECT: (no value), SparkFun-Switches:SWITCH-SPDT-PTH-11.6X4.0MM-LOCK
- 3.3/5VOUT: device SparkFun-Connectors:CONN_03SCREW_LOCK -> SparkFun-Connectors:CONN_03-SCREW-5MM
Connections:
- new net IR1RAW: 7R2.1, 7UP-R1.2, IR/OUT.1, U1.OUT
- new net IR2RAW: 7R4.1, 7UP-R2.2, IR/OUT.3, U2.OUT
- new net N$34: 7C1.2, 7R1.2, U1.VS
- new net N$35: 7R1.1, 7R3.1, 7UP-R1.1, 7UP-R2.1, VSELECT.P
- new net N$41: 7C2.1, 7R2.2, IR/OUT.2
- new net N$43: 7C3.2, 7R3.2, U2.VS
- new net N$44: 7C4.1, 7R4.2, IR/OUT.4
- net 0: now also STM32OUT1.19; no longer STM32OUT1.20
- net 1: now also STM32OUT1.18; no longer STM32OUT1.19
- net 2: now also STM32OUT1.17; no longer STM32OUT1.18
- net 3.3V: now also VSELECT.O
- net 5V: now also VSELECT.S
- net GND: now also 7C1.1, 7C2.2, 7C3.1, 7C4.2, CAPACITOR.3, U1.GND, U2.GND; no longer CAPACITOR.1
- net N$32: now also MOTOROUT.1; no longer MOTOROUT.3
- net N$33: now also MOTOROUT.3; no longer MOTOROUT.1
- net VCC_1: now also CAPACITOR.1; no longer CAPACITOR.3

Commit message: 16/12 PCB shit too much happened shld have committed more often but wtv deleted stm32 sheet added IR and mouse sensor Finally routed everything, gerber files are included hopefully done for now
Parts:
- removed 5C1, 5C2: 18pF, rcl:C-EUC0603
- removed 5C10, 5C5, 5C7, 5C8, 5C9: 1uF, rcl:C-EUC0603
- removed 5C3, 5C4: 47pF, rcl:C-EUC0603
- removed 5C6: 1uf, rcl:C-EUC0603
- removed 5D1: SS14, diode:DIODE-DO-214AC
- removed 5DOWN-R1, 5R3, 5R4: 22, rcl:R-EU_R0603
- removed 5F1: 300ohm bead, rcl:R-EU_R0402
- removed 5LED1: RED, SparkFun-LED:LED-RED1206
- removed 5OSC: 8MHz, SparkFun-Clocks:CRYSTALSMD-HC49UP
- removed 5R1, 5R5: 1k, rcl:R-EU_R0603
- removed 5R2, 5R6: 10k, rcl:R-EU_R0603
- removed 5RESET: TAC_SWITCHSMD, SparkFun-Retired:TAC_SWITCHSMD
- removed 5UP-R1: 1.5k, rcl:R-EU_R0603
- removed BOOT-JUMPER: (no value), SparkFun-Connectors:CONN_03LOCK
- removed STM32OUT1, STM32OUT2: (no value), SparkFun-Connectors:CONN_20LOCK
- removed U$7: AMS1117-3.3, SparkFun-IC-Power:V_REG_LD1117VXXLD1117-SMD
- removed U1, U2: 38kHz, SparkFun-Sensors:TSOP38238
- removed UC1: STM32F103CBT6, stm32:STM32F103CB
- removed VREGJUMPER: (no value), SparkFun-Connectors:CONN_02LOCK
- removed X1: USB-MINIB, SparkFun-Connectors:USB_MINI-B_SMT
- added C1, C2: 1.0uF, SparkFun-Capacitors:1.0UF-0603-16V-10%-X7R
- added C3: 0.1uF, SparkFun-Capacitors:0.1UF-0603-25V-5%
- added C4: 4.7uF, SparkFun-Capacitors:4.7UF-0603-6.3V-(10%)
- added IR1, IR2: 38kHz, SparkFun-Sensors:TSOP38238
- added J1: (no value), SparkFun-Connectors:CONN_06LOCK
- added R1: 39, SparkFun-Resistors:RESISTOR0603
- added R2, R3: 10k, SparkFun-Resistors:10KOHM-0603-1/10W-1%
- added U$1: LN6206, MCP1700T-3302E_TT:MCP1700T-3302E/TT
- added U$2: PMW3360, JH:PMW3360
- DRIVER-IO: device SparkFun-Connectors:CONN_06LOCK -> SparkFun-Connectors:CONN_07LOCK
Connections:
- removed net 0: STM32OUT1.19, UC1.PB11/I2C2_SDA/USART3_RX
- removed net 1: STM32OUT1.18, UC1.PB10/I2C2_SCL/USART3_TX
- removed net 10: STM32OUT1.9, UC1.PA1/USART2_RTS/ADC12_IN1/TIM2_CH2
- removed net 11: STM32OUT1.8, UC1.PA0_WKUP/USART2_CTS/ADC12_IN0/TIM2_CH1_ETR
- removed net 12: STM32OUT1.6, UC1.PC15-OSC32_OUT
- removed net 13: STM32OUT1.5, UC1.PC14-OSC32_IN
- removed net 14: STM32OUT1.4, UC1.PC13-TAMPER-RTC
- removed net 15: STM32OUT2.17, UC1.PB7/I2C1_SDA/TIM4_CH2
- removed net 16: STM32OUT2.16, UC1.PB6/I2C1_SCL/TIM4_CH1
- removed net 17: STM32OUT2.15, UC1.PB5/I2C1_SMBA
- removed net 18: STM32OUT2.14, UC1.PB4/NJTRST
- removed net 19: STM32OUT2.13, UC1.PB3/JTDO
- removed net 2: STM32OUT1.17, UC1.PB2/BOOT1
- removed net 20: STM32OUT2.12, UC1.PA15/JTDI
- removed net 21: STM32OUT2.11, UC1.PA14/JTCK/SWCLK
- removed net 22: STM32OUT2.10, UC1.PA13/JTMS/SWDIO
- removed net 23_USBDP: 5C4.2, 5R4.1, 5UP-R1.1, STM32OUT2.9, UC1.PA12/USART1_RTS/CAN_TX/TIM1_ETR/USBDP
- removed net 24_USBDM: 5C3.2, 5R3.1, STM32OUT2.8, UC1.PA11/USART1_CTS/CAN_RX/TIM1_CH4/USBDM
- removed net 25: STM32OUT2.7, UC1.PA10/USART1_RX/TIM1_CH3
- removed net 26: STM32OUT2.6, UC1.PA9/USART1_TX/TIM1_CH2
- removed net 27: STM32OUT2.5, UC1.PA8/USART1_CK/TIM1_CH1/MCO
- removed net 28: STM32OUT2.4, UC1.PB15/SPI2_MOSI/TIM1_CH3N
- removed net 29: STM32OUT2.3, UC1.PB14/SPI2_MISO/USART3_RTS/TIM1_CH2N
- removed net 3: STM32OUT1.16, UC1.PB0/ADC12_IN8/TIM3_CH3
- removed net 30: STM32OUT2.2, UC1.PB13/SPI2_SCK/USART3_CTS/TIM1_CH1N
- removed net 31: STM32OUT2.1, UC1.PB12/SPI2_NSS/I2C2_SMBA/USART3_CK/TIM1_BKIN
- removed net 32: 5R6.1, STM32OUT2.18, UC1.BOOT0, UC1.PB8/TIM4_CH3
- removed net 4: STM32OUT1.15, UC1.PA7/SPI1_MOSI/ADC12_IN7/TIM3_CH2
- removed net 5: STM32OUT1.14, UC1.PA6/SPI1_MISO/ADC12_IN6/TIM3_CH1
- removed net 6: STM32OUT1.13, UC1.PA5/SPI1_SCK/ADC12_IN5
- removed net 7: STM32OUT1.12, UC1.PA4/SPI1_NSS/USART2_CK/ADC12_IN4
- removed net 8: STM32OUT1.11, UC1.PA3/USART2_RX/ADC12_IN3/TIM2_CH4
- removed net 9: STM32OUT1.10, UC1.PA2/USART2_TX/ADC12_IN2/TIM2_CH3
- removed net AGND: 5C10.2, 5F1.1, STM32OUT1.7, UC1.VSS_A
- removed net DISC: UC1.PB9/TIM4_CH4
- removed net N$18: U$7.IN, VREGJUMPER.2
- removed net N$27: 5R1.2, 5RESET.1, 5RESET.2
- removed net N$28: 5LED1.A, 5R5.1
- removed net N$30: 5R6.2, BOOT-JUMPER.2
- removed net N$31: 5R5.2, UC1.PB1/ADC12_IN9/TIM3_CH4
- removed net N$59: 5R3.2, X1.D-
- removed net N$60: 5R4.2, X1.D+
- removed net OSC_IN: 5C2.1, 5OSC.2, UC1.PD0-OSC_IN
- removed net OSC_OUT: 5C1.1, 5OSC.1, UC1.PD1-OSC_OUT
- removed net RESET: 5R2.1, 5RESET.3, 5RESET.4, UC1.NRST
- removed net VBAT: STM32OUT1.3, UC1.VBAT
- removed net V_USB: 5D1.A, X1.VBUS
- new net 1.8V: C1.1, R1.2, U$1.VOUT, U$2.VDD
- new net N$40: J1.6, U$2.NCS
- new net N$42: J1.5, R2.1, U$2.MISO
- new net N$45: J1.4, U$2.MOSI
- new net N$46: J1.3, U$2.SCLK
- new net N$47: J1.2, U$2.MOT
- new net N$48: C3.2, C4.2, U$2.VDDPIX
- new net NRESET: J1.1, R3.2, U$2.NRESET
- net 3.3V: now also C2.1, R2.2, R3.1, U$1.VIN, U$2.VDDIO; no longer 5C10.1, 5C6.1, 5C7.1, 5C8.1, 5C9.1, 5R2.2, 5UP-R1.2, BOOT-JUMPER.1, U$7.OUT, UC1.VDD_1, UC1.VDD_2, UC1.VDD_3, UC1.VDD_A
- net 5V: no longer 5C5.1, 5D1.C, VREGJUMPER.1
- net GND: now also C1.2, C2.2, C3.1, C4.1, IR1.GND, IR2.GND, U$1.GND, U$2.GND; no longer 5C1.2, 5C2.2, 5C3.1, 5C4.1, 5C5.2, 5C6.2, 5C7.2, 5C8.2, 5C9.2, 5DOWN-R1.1, 5F1.2, 5LED1.C, 5R1.1, BOOT-JUMPER.3, U$7.GND, U1.GND, U2.GND, UC1.VSS_1, UC1.VSS_2, UC1.VSS_3, X1.GND
- net IR1RAW: now also IR1.OUT; no longer U1.OUT
- net IR2RAW: now also IR2.OUT; no longer U2.OUT
- net N$34: now also IR1.VS; no longer U1.VS
- net N$36: now also R1.1, U$2.LED_P; no longer 5DOWN-R1.2, X1.SHIELD
- net N$43: now also IR2.VS; no longer U2.VS
- net SOLENOIDON: now also DRIVER-IO.7
Other:
- note removed: "BOOT0"
