File: PCB/projects/PCB1_v1/PCB1_v1.sch (EAGLE design)
At the start: 12 parts

Commit message: 24/2 PCB v0.2 Finished new VNH5019 Motor Driver circuit, step up/down + solenoid, left with light sensors (+MUX+Comparators) and other sensors and connections. lesgo
Parts:
- added 3C1: 100uF, SparkFun-Capacitors:100UF-POLAR-25V-20%(ELEC)
- added 3C10, 3C11: 22.0uF, rcl:C-EUC1210
- added 3C12: 10.0nF, rcl:C-EUC0603
- added 3C13: 470uF, rcl:CPOL-USD/7343-31R
- added 3C2: 680nF, SparkFun-Capacitors:680PF-0603-50V-10%
- added 3C3: 0.1uF, SparkFun-Capacitors:0.1UF-0603-25V-5%
- added 3C4, 3C5: 1000uF, JH:1000UF-CAP
- added 3C6, 3C7: 1500pF, rcl:C-EUC0603
- added 3C8: 22UF, SparkFun-Capacitors:22UF-1210-16V-20%
- added 3C9: 6.8uF, rcl:CPOL-USA/3216-18R
- added 3D1: SS510, diode:SCHOTTKY-DIODESMD
- added 3D2, 3D4: 1N4728, diode:1N4728
- added 3D3, 3D5: 1N5401, diode:1N5400
- added 3D6, 3D7: SS54, diode:SCHOTTKY-DIODESMD
- added 3J1, 3J2, J1M1, J1M2, J1M3, J1M4: (no value), SparkFun-Connectors:CONN_03-SCREW-5MM
- added 3L1: 100UH-L, JH:100UH-L
- added 3L2: 33uH, JH:CDRH127
- added 3L3: XAL6060/10uH, JH:XAL6060
- added 3Q1, 3Q3: STP75NF75, SparkFun-DiscreteSemi:MOSFET-NCH-FQP30N06L
- added 3Q2, 3Q4: AO3400, SparkFun-DiscreteSemi:MOSFET-NCH-AO3404A
- added 3R1: 2.94k, SparkFun-Resistors:RESISTOR0603
- added 3R10, 3R5: 20, rcl:R-EU_R0603
- added 3R11, 3R4, 3R6, 3R8, 3R9: 10k, rcl:R-EU_R0603
- added 3R12: 5.9k, rcl:R-EU_R0603
- added 3R2: 2.0k, SparkFun-Resistors:2.0KOHM-0603-1/10W-5%
- added 3R3, 3R7: 1k, rcl:R-EU_R0603
- added 3U1: LM2587, JH:LM2587
- added 3U2: (no value), JH:MCP41XXX
- added 4U1: LM2596, JH:LM2596
- added 4U2: 3.1v, JH:TPS5450
- added C1M1, C1M2, C1M3, C1M4: 33nF, SparkFun-Capacitors:33NF-0603-50V-10%
- added C2M1, C2M2, C2M3, C2M4: 680uF, rcl:CPOL-USE3.5-8
- added C3M1, C3M2, C3M3, C3M4: 1.0uF, SparkFun-Capacitors:1.0UF-0603-16V-10%-X7R
- added D12M1, D12M2, D12M3, D12M4: 4.7k, SparkFun-Resistors:4.7KOHM-0603-1/10W-1%
- added D1M1, D1M2, D1M3, D1M4: GREEN, SparkFun-LED:LED-GREEN1206
- added D2M1, D2M2, D2M3, D2M4: RED, SparkFun-LED:LED-RED1206
- added Q1M1, Q1M2, Q1M3, Q1M4: AOD482, SparkFun-DiscreteSemi:MOSFET-NCH-FDD8780
- added R10M1, R10M2, R10M3, R10M4, R3M1, R3M2, R3M3, R3M4, R4M1, R4M2, R4M3, R4M4, R5M1, R5M2, R5M3, R5M4, R6M1, R6M2, R6M3, R6M4, R7M1, R7M2, R7M3, R7M4: 1k, SparkFun-Resistors:1KOHM-0603-1/10W-1%
- added R11M1, R11M2, R11M3, R11M4, R8M1, R8M2, R8M3, R8M4, R9M1, R9M2, R9M3, R9M4: 10k, SparkFun-Resistors:10KOHM-0603-1/10W-1%
- added R1M1, R1M2, R1M3, R1M4, R2M1, R2M2, R2M3, R2M4: 3.3k, SparkFun-Resistors:3.3KOHM-0603-1/10W-1%
- added U1M1, U1M2, U1M3, U1M4: VNH5019, JH:VNH5019
Connections:
- new net 12V: 3C1.+, 3C10.1, 3C11.1, 3C8.1, 3L1.1, 3R3.1, 3R4.2, 3R7.1, 3R8.2, 3U1.VIN, 4U1.VIN, 4U2.VIN, Q1M1.S, Q1M2.S, Q1M3.S, Q1M4.S, U1M1.VBAT, U1M2.VBAT, U1M3.VBAT, U1M4.VBAT
- new net 5V: 3C9.+, 3L2.2, 4U1.FDBK
- new net CPM1: Q1M1.G, U1M1.CP
- new net CPM2: Q1M2.G, U1M2.CP
- new net CPM3: Q1M3.G, U1M3.CP
- new net CPM4: Q1M4.G, U1M4.CP
- new net CSDIS: R9M1.1, R9M2.1, R9M3.1, R9M4.1, U1M1.CS_DIS, U1M2.CS_DIS, U1M3.CS_DIS, U1M4.CS_DIS
- new net CSM1: C1M1.2, R8M1.1
- new net CSM2: C1M2.2, R8M2.1
- new net CSM3: C1M3.2, R8M3.1
- new net CSM4: C1M4.2, R8M4.1
- new net CS_POT: 3U2.CS
- new net ENAM1: R3M1.1
- new net ENAM2: R3M2.1
- new net ENAM3: R3M3.1
- new net ENAM4: R3M4.1
- new net ENBM1: R4M1.2
- new net ENBM2: R4M2.2
- new net ENBM3: R4M3.2
- new net ENBM4: R4M4.2
- new net INAM1: R5M1.1
- new net INAM2: R5M2.1
- new net INAM3: R5M3.1
- new net INAM4: R5M4.1
- new net INBM1: R6M1.2
- new net INBM2: R6M2.2
- new net INBM3: R6M3.2
- new net INBM4: R6M4.2
- new net MOSI_POT: 3U2.MOSI
- new net N$10: R2M2.1, R3M2.2, U1M2.EN_A
- new net N$11: R5M2.2, U1M2.IN_A
- new net N$12: D12M1.1, D1M1.C, D2M1.A
- new net N$13: R1M2.1, R4M2.1, U1M2.EN_B
- new net N$14: R6M2.1, U1M2.IN_B
- new net N$15: R10M2.2, R8M2.2, U1M2.CS
- new net N$16: R7M2.1, U1M2.PWM_IN
- new net N$17: D12M2.1, D1M2.C, D2M2.A
- new net N$18: C2M3.+, C3M3.1, Q1M3.D, U1M3.VCC
- new net N$19: R2M3.1, R3M3.2, U1M3.EN_A
- new net N$2: R2M1.1, R3M1.2, U1M1.EN_A
- new net N$20: R5M3.2, U1M3.IN_A
- new net N$21: R1M3.1, R4M3.1, U1M3.EN_B
- new net N$22: R6M3.1, U1M3.IN_B
- new net N$23: R10M3.2, R8M3.2, U1M3.CS
- new net N$24: R7M3.1, U1M3.PWM_IN
- new net N$25: D12M3.1, D1M3.C, D2M3.A
- new net N$26: C2M4.+, C3M4.1, Q1M4.D, U1M4.VCC
- new net N$27: R2M4.1, R3M4.2, U1M4.EN_A
- new net N$28: R5M4.2, U1M4.IN_A
- new net N$29: R1M4.1, R4M4.1, U1M4.EN_B
- new net N$3: C2M1.+, C3M1.1, Q1M1.D, U1M1.VCC
- new net N$30: R6M4.1, U1M4.IN_B
- new net N$31: R10M4.2, R8M4.2, U1M4.CS
- new net N$32: R7M4.1, U1M4.PWM_IN
- new net N$33: D12M4.1, D1M4.C, D2M4.A
- new net N$34: 3D1.A, 3L1.2, 3U1.SW
- new net N$35: 3C6.2, 3Q1.S, 3Q2.D, 3R4.1
- new net N$36: 3R1.2, 3U1.COMP
- new net N$37: 3C2.1, 3R1.1
- new net N$38: 3Q1.G, 3R3.2
- new net N$39: 3D2.C, 3D3.C
- new net N$4: R1M1.1, R4M1.1, U1M1.EN_B
- new net N$40: 3C6.1, 3R5.1
- new net N$41: 3U2.PA0, 3U2.PW0
- new net N$42: 3C7.2, 3Q3.S, 3Q4.D, 3R8.1
- new net N$43: 3Q3.G, 3R7.2
- new net N$44: 3D4.C, 3D5.C
- new net N$45: 3C7.1, 3R10.1
- new net N$46: 3C12.1, 4U2.BOOT
- new net N$47: 3D6.C, 3L2.1, 4U1.OUT
- new net N$48: 3C12.2, 3D7.C, 3L3.1, 4U2.PH
- new net N$49: 3R11.1, 3R12.2, 4U2.VSNS
- new net N$5: R6M1.1, U1M1.IN_B
- new net N$6: R5M1.2, U1M1.IN_A
- new net N$7: R10M1.2, R8M1.2, U1M1.CS
- new net N$8: R7M1.1, U1M1.PWM_IN
- new net N$9: C2M2.+, C3M2.1, Q1M2.D, U1M2.VCC
- new net OUTAM1: D1M1.A, D2M1.C, J1M1.1, U1M1.OUT_A
- new net OUTAM2: D1M2.A, D2M2.C, J1M2.1, U1M2.OUT_A
- new net OUTAM3: D1M3.A, D2M3.C, J1M3.1, U1M3.OUT_A
- new net OUTAM4: D1M4.A, D2M4.C, J1M4.1, U1M4.OUT_A
- new net OUTBM1: D12M1.2, J1M1.3, U1M1.OUT_B
- new net OUTBM2: D12M2.2, J1M2.3, U1M2.OUT_B
- new net OUTBM3: D12M3.2, J1M3.3, U1M3.OUT_B
- new net OUTBM4: D12M4.2, J1M4.3, U1M4.OUT_B
- new net PWMM1: R11M1.2, R7M1.2
- new net PWMM2: R11M2.2, R7M2.2
- new net PWMM3: R11M3.2, R7M3.2
- new net PWMM4: R11M4.2, R7M4.2
- new net SCLK_POT: 3U2.SCLK
- new net SOLENOID-: 3D3.A, 3J1.3, 3Q1.D, 3R5.2
- new net SOLENOID-1: 3D5.A, 3J2.3, 3Q3.D, 3R10.2
- new net SOLENOIDON1: 3Q2.G, 3R6.2
- new net SOLENOIDON2: 3Q4.G, 3R9.2
- new net VCC_2: 3C4.+, 3C5.+, 3D1.C, 3D2.A, 3D4.A, 3J1.1, 3J2.1, 3R2.2, 3U1.FDBK, 3U2.PB0
- net 3.3V: now also 3C13.+, 3C3.1, 3L3.2, 3R11.2, 3U2.VCC, R1M1.2, R1M2.2, R1M3.2, R1M4.2, R2M1.2, R2M2.2, R2M3.2, R2M4.2
- net GND: now also 3C1.-, 3C10.2, 3C11.2, 3C13.-, 3C2.2, 3C3.2, 3C4.-, 3C5.-, 3C8.2, 3C9.-, 3D6.A, 3D7.A, 3Q2.S, 3Q4.S, 3R12.1, 3R2.1, 3R6.1, 3R9.1, 3U1.GND, 3U2.GND, 4U1.ENA, 4U1.GND, 4U2.GND, C1M1.1, C1M2.1, C1M3.1, C1M4.1, C2M1.-, C2M2.-, C2M3.-, C2M4.-, C3M1.2, C3M2.2, C3M3.2, C3M4.2, R10M1.1, R10M2.1, R10M3.1, R10M4.1, R11M1.1, R11M2.1, R11M3.1, R11M4.1, R9M1.2, R9M2.2, R9M3.2, R9M4.2, U1M1.GND, U1M2.GND, U1M3.GND, U1M4.GND
