File: PCB/projects/PCB2k19/PCB1.brd (EAGLE design)
At the start: 190.7 x 218 mm, 265 parts, among them Q1M1 AOD482, Q1M2 AOD482, Q1M3 AOD482, Q1M4 AOD482, U1M1 VNH5019, U1M2 VNH5019, U1M3 VNH5019, U1M4 VNH5019

Commit message: 17/3 Updated derp in Boost Circuit voltage selection, updated boards even further
Parts:
- removed 1PT0, 1PT1, 1PT10, 1PT11, 1PT12, 1PT13, 1PT14, 1PT15, 1PT16, 1PT17, 1PT18, 1PT19, 1PT2, 1PT20, 1PT21, 1PT22, 1PT23, 1PT24, 1PT25, 1PT26, 1PT27, 1PT28, 1PT29, 1PT3, 1PT30, 1PT31, 1PT32, 1PT33, 1PT34, 1PT35, 1PT36, 1PT37, 1PT38, 1PT39, 1PT4, 1PT40, 1PT41, 1PT42, 1PT43, 1PT44, 1PT45, 1PT46, 1PT47, 1PT5, 1PT6, 1PT7, 1PT8, 1PT9: TEMT6000, SparkFun-Sensors:TEMT6000
- removed D12M1: 4.7k, SparkFun-Resistors:0603
- added PT0, PT1, PT10, PT11, PT12, PT13, PT14, PT15, PT16, PT17, PT18, PT19, PT2, PT20, PT21, PT22, PT23, PT24, PT25, PT26, PT27, PT28, PT29, PT3, PT30, PT31, PT32, PT33, PT34, PT35, PT36, PT37, PT38, PT39, PT4, PT40, PT41, PT42, PT43, PT44, PT45, PT46, PT47, PT5, PT6, PT7, PT8, PT9: TEMT6000, SparkFun-Sensors:TEMT6000
- added R12M1: 4.7k, SparkFun-Resistors:0603
- 1R10, 1R11, 1R2, 1R5, 1R8, 3R10, 3R11, 3R12, 3R3, 3R4, 3R5, 3R6, 3R7, 3R8, 3R9: device rcl:R0603 -> SparkFun-Resistors:0603
- 3C10, 3C11: device rcl:C1210 -> SparkFun-Capacitors:1210
- 3C12: value 10.0nF -> 10nF; device rcl:C0603 -> SparkFun-Capacitors:0603
- 3C6, 3C7: device rcl:C0603 -> SparkFun-Capacitors:0603
- 3R2: value 2.0k -> 1.69k
- moved R10M1 321.7 mm to (89.5, 115.7), turned to 180 degrees
- moved R3M1 319.4 mm to (81.9, 119.5), turned to 270 degrees
- moved R2M1 309.8 mm to (89.5, 108.1)
- moved R9M1 306.3 mm to (89.5, 113.1)
- moved R1M1 295.3 mm to (89.5, 110.6)
- moved U1M1 294.8 mm to (78.1, 106.8), turned to 180 degrees
- moved IRIN2 290.3 mm to (54.6, -31.8), turned to 90 degrees
- moved LED43 289.2 mm to (67.3, 2.54), flipped to the bottom, turned to 180 degrees
- moved 1R13 288.3 mm to (50.8, -31.8), flipped to the bottom, turned to 180 degrees
- moved Q1M1 284.6 mm to (64.1, 114.4), turned to 180 degrees
- moved R8M1 280.1 mm to (76.8, 119.5), turned to 270 degrees
- moved LED42 276.5 mm to (59.7, 2.54), flipped to the bottom, turned to 180 degrees
- moved R7M1 267.7 mm to (79.3, 119.5), turned to 90 degrees
- moved LED23 263.4 mm to (31.0, -37.0), flipped to the bottom, turned to 50 degrees
- moved LED22 263.0 mm to (37.0, -31.0), flipped to the bottom, turned to 40 degrees
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- renumbered D12M2 to R12M2, D12M3 to R12M3, D12M4 to R12M4
Connections:
- removed net N$104: 1PT47.EMITTER, 1U4.P16
- removed net N$41: 3U2.5, 3U2.6
- new net N$68: 1U3.P9, PT16.EMITTER
- new net N$69: 1U3.P8, PT17.EMITTER
- net 12V: now also J6.1; no longer 3C1.+, 3L1.P1, 3R3.1, 3R4.2, 3R7.1, 3R8.2, 3U1.P5, J6.3
- net 3.3V: now also PT0.COLLECTOR, PT1.COLLECTOR, PT10.COLLECTOR, PT11.COLLECTOR, PT12.COLLECTOR, PT13.COLLECTOR, PT14.COLLECTOR, PT15.COLLECTOR, PT16.COLLECTOR, PT17.COLLECTOR, PT18.COLLECTOR, PT19.COLLECTOR, PT2.COLLECTOR, PT20.COLLECTOR, PT21.COLLECTOR, PT22.COLLECTOR, PT23.COLLECTOR, PT24.COLLECTOR, PT25.COLLECTOR, PT26.COLLECTOR, PT27.COLLECTOR, PT28.COLLECTOR, PT29.COLLECTOR, PT3.COLLECTOR, PT30.COLLECTOR, PT31.COLLECTOR, PT32.COLLECTOR, PT33.COLLECTOR, PT34.COLLECTOR, PT35.COLLECTOR, PT36.COLLECTOR, PT37.COLLECTOR, PT38.COLLECTOR, PT39.COLLECTOR, PT4.COLLECTOR, PT40.COLLECTOR, PT41.COLLECTOR, PT42.COLLECTOR, PT43.COLLECTOR, PT44.COLLECTOR, PT45.COLLECTOR, PT46.COLLECTOR, PT47.COLLECTOR, PT5.COLLECTOR, PT6.COLLECTOR, PT7.COLLECTOR, PT8.COLLECTOR, PT9.COLLECTOR; no longer 1PT0.COLLECTOR, 1PT1.COLLECTOR, 1PT10.COLLECTOR, 1PT11.COLLECTOR, 1PT12.COLLECTOR, 1PT13.COLLECTOR, 1PT14.COLLECTOR, 1PT15.COLLECTOR, 1PT16.COLLECTOR, 1PT17.COLLECTOR, 1PT18.COLLECTOR, 1PT19.COLLECTOR, 1PT2.COLLECTOR, 1PT20.COLLECTOR, 1PT21.COLLECTOR, 1PT22.COLLECTOR, 1PT23.COLLECTOR, 1PT24.COLLECTOR, 1PT25.COLLECTOR, 1PT26.COLLECTOR, 1PT27.COLLECTOR, 1PT28.COLLECTOR, 1PT29.COLLECTOR, 1PT3.COLLECTOR, 1PT30.COLLECTOR, 1PT31.COLLECTOR, 1PT32.COLLECTOR, 1PT33.COLLECTOR, 1PT34.COLLECTOR, 1PT35.COLLECTOR, 1PT36.COLLECTOR, 1PT37.COLLECTOR, 1PT38.COLLECTOR, 1PT39.COLLECTOR, 1PT4.COLLECTOR, 1PT40.COLLECTOR, 1PT41.COLLECTOR, 1PT42.COLLECTOR, 1PT43.COLLECTOR, 1PT44.COLLECTOR, 1PT45.COLLECTOR, 1PT46.COLLECTOR, 1PT47.COLLECTOR, 1PT5.COLLECTOR, 1PT6.COLLECTOR, 1PT7.COLLECTOR, 1PT8.COLLECTOR, 1PT9.COLLECTOR
- net N$1: now also PT0.EMITTER; no longer 1PT0.EMITTER
- net N$100: now also 1U4.P18, PT45.EMITTER; no longer 1PT43.EMITTER, 1U4.P20
- net N$101: now also 1U4.P17, PT46.EMITTER; no longer 1PT44.EMITTER, 1U4.P19
- net N$102: now also 1U4.P16, PT47.EMITTER; no longer 1PT45.EMITTER, 1U4.P18
- net N$103: now also 3R2.2, 3U1.P2, 3U2.7; no longer 1PT46.EMITTER, 1U4.P17
- net N$12: now also R12M1.1; no longer D12M1.1
- net N$51: now also PT1.EMITTER; no longer 1PT1.EMITTER
- net N$52: now also PT2.EMITTER; no longer 1PT2.EMITTER
- net N$53: now also PT3.EMITTER; no longer 1PT3.EMITTER
- net N$54: now also PT4.EMITTER; no longer 1PT4.EMITTER
- net N$55: now also PT5.EMITTER; no longer 1PT5.EMITTER
- net N$56: now also PT6.EMITTER; no longer 1PT6.EMITTER
- net N$57: now also PT7.EMITTER; no longer 1PT7.EMITTER
- net N$58: now also PT8.EMITTER; no longer 1PT8.EMITTER
- net N$59: now also PT9.EMITTER; no longer 1PT9.EMITTER
- net N$60: now also PT10.EMITTER; no longer 1PT10.EMITTER
- net N$61: now also PT11.EMITTER; no longer 1PT11.EMITTER
- net N$62: now also PT12.EMITTER; no longer 1PT12.EMITTER
- net N$63: now also PT13.EMITTER; no longer 1PT13.EMITTER
- net N$64: now also PT14.EMITTER; no longer 1PT14.EMITTER
- net N$65: now also PT15.EMITTER; no longer 1PT15.EMITTER
- net N$71: now also 1U3.P7, PT18.EMITTER; no longer 1PT16.EMITTER, 1U3.P9
- net N$72: now also 1U3.P6, PT19.EMITTER; no longer 1PT17.EMITTER, 1U3.P8
- net N$73: now also 1U3.P5, PT20.EMITTER; no longer 1PT18.EMITTER, 1U3.P7
- net N$74: now also 1U3.P4, PT21.EMITTER; no longer 1PT19.EMITTER, 1U3.P6
- net N$75: now also 1U3.P3, PT22.EMITTER; no longer 1PT20.EMITTER, 1U3.P5
- net N$76: now also 1U3.P2, PT23.EMITTER; no longer 1PT21.EMITTER, 1U3.P4
- net N$77: now also 1U3.P23, PT24.EMITTER; no longer 1PT22.EMITTER, 1U3.P3
- net N$78: now also 1U3.P22, PT25.EMITTER; no longer 1PT23.EMITTER, 1U3.P2
- net N$79: now also 1U3.P21, PT26.EMITTER; no longer 1PT24.EMITTER, 1U3.P23
- net N$80: now also 1U3.P20, PT27.EMITTER; no longer 1PT25.EMITTER, 1U3.P22
- net N$81: now also 1U3.P19, PT28.EMITTER; no longer 1PT26.EMITTER, 1U3.P21
- net N$82: now also 1U3.P18, PT29.EMITTER; no longer 1PT27.EMITTER, 1U3.P20
- net N$83: now also 1U3.P17, PT30.EMITTER; no longer 1PT28.EMITTER, 1U3.P19
- net N$84: now also 1U3.P16, PT31.EMITTER; no longer 1PT29.EMITTER, 1U3.P18
- net N$85: now also 1U4.P9, PT32.EMITTER; no longer 1PT30.EMITTER, 1U3.P17
- net N$86: now also 1U4.P8, PT33.EMITTER; no longer 1PT31.EMITTER, 1U3.P16
- net N$89: now also 1U4.P7, PT34.EMITTER; no longer 1PT32.EMITTER, 1U4.P9
- net N$90: now also 1U4.P6, PT35.EMITTER; no longer 1PT33.EMITTER, 1U4.P8
- net N$91: now also 1U4.P5, PT36.EMITTER; no longer 1PT34.EMITTER, 1U4.P7
- net N$92: now also 1U4.P4, PT37.EMITTER; no longer 1PT35.EMITTER, 1U4.P6
- net N$93: now also 1U4.P3, PT38.EMITTER; no longer 1PT36.EMITTER, 1U4.P5
- net N$94: now also 1U4.P2, PT39.EMITTER; no longer 1PT37.EMITTER, 1U4.P4
- net N$95: now also 1U4.P23, PT40.EMITTER; no longer 1PT38.EMITTER, 1U4.P3
- net N$96: now also 1U4.P22, PT41.EMITTER; no longer 1PT39.EMITTER, 1U4.P2
- net N$97: now also 1U4.P21, PT42.EMITTER; no longer 1PT40.EMITTER, 1U4.P23
- net N$98: now also 1U4.P20, PT43.EMITTER; no longer 1PT41.EMITTER, 1U4.P22
- net N$99: now also 1U4.P19, PT44.EMITTER; no longer 1PT42.EMITTER, 1U4.P21
- net OUTBM1: now also R12M1.2; no longer D12M1.2
- net VCC_1: now also 3C1.+, 3L1.P1, 3R3.1, 3R4.2, 3R7.1, 3R8.2, 3U1.P5, J6.3; no longer J6.1
- net VCC_2: now also 3U2.5, 3U2.6; no longer 3R2.2, 3U1.P2, 3U2.7
Routing:
- added copper zone on layer 1, net GND
- added copper zone on layer 16, net GND

Commit message: 18/3 Moved boost circuit and solenoid circuits to PCB2 else no space
Parts:
- removed 3C1: 100uF, SparkFun-Capacitors:PANASONIC_D
- removed 3C2: 680nF, SparkFun-Capacitors:0603
- removed 3C3: 0.1uF, SparkFun-Capacitors:0603
- removed 3C4, 3C5: 1000uF, JH:1000UF-CAP
- removed 3C6, 3C7: 1500pF, SparkFun-Capacitors:0603
- removed 3C8: 22UF, SparkFun-Capacitors:1210
- removed 3C9: 6.8uF, rcl:A/3216-18R
- removed 3D1: SS510, diode:SMB
- removed 3D2, 3D4: 1N4728, diode:DO41Z10
- removed 3D3, 3D5: 1N5401, diode:DO201-15
- removed 3D6: SS54, diode:SMB
- removed 3J1, 3J2: (no value), SparkFun-Connectors:SCREWTERMINAL-5MM-3
- removed 3L1: 100UH-L, JH:100UH-L
- removed 3L2: 33uH, JH:127
- removed 3Q1, 3Q3: STP75NF75, SparkFun-DiscreteSemi:TO220V
- removed 3Q2, 3Q4: AO3400, SparkFun-DiscreteSemi:SOT23-3
- removed 3R1: 2.94k, SparkFun-Resistors:0603
- removed 3R10, 3R5: 20, SparkFun-Resistors:0603
- removed 3R2: 1.69k, SparkFun-Resistors:0603
- removed 3R3, 3R7: 1k, SparkFun-Resistors:0603
- removed 3R4, 3R6, 3R8, 3R9: 10k, SparkFun-Resistors:0603
- removed 3U1: LM2587, JH:TO-263
- removed 3U2: (no value), JH:SOIC-8
- removed 4U1: LM2596, JH:TO-263
- removed J3: (no value), SparkFun-Connectors:SCREWTERMINAL-3.5MM-3_LOCK.007S
- removed J7: (no value), SparkFun-Connectors:1X04_LOCK
- J2, J4, J5, J6: device SparkFun-Connectors:SCREWTERMINAL-3.5MM-3_LOCK.007S -> SparkFun-Connectors:SCREWTERMINAL-5MM-3
- moved 3C10 302.2 mm to (2.54, 2.54)
- moved 3C11 302.2 mm to (6.35, 2.54)
- moved 3D7 302.2 mm to (7.62, -3.81)
- moved 3R11 302.2 mm to (20.3, 3.81)
- moved 3R12 302.2 mm to (20.3, 0.00)
- moved 4U2 302.2 mm to (14.0, 2.54)
- moved 3C12 301.9 mm to (14.0, -3.81)
- moved 3L3 298.4 mm to (15.2, 10.2), turned to 90 degrees
- moved 3C13 297.2 mm to (5.08, 10.2)
- moved R10M3 289.7 mm to (35.4, -44.2), turned to 135 degrees
- moved R9M3 274.0 mm to (32.7, -46.9), turned to 315 degrees
- moved R2M3 273.2 mm to (27.4, -52.3), turned to 315 degrees
- moved R10M2 262.9 mm to (31.5, 48.1), turned to 225 degrees
- moved R1M3 260.6 mm to (30.0, -49.6), turned to 315 degrees
- moved R2M2 259.8 mm to (39.6, 40.1), turned to 45 degrees
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Connections:
- removed net 5V: 3C9.+, 3L2.2, 4U1.P4, J2.2
- removed net CS_POT: 3U2.1, J1.15
- removed net MOSI_POT: 3U2.3, J1.19
- removed net N$103: 3R2.2, 3U1.P2, 3U2.7
- removed net N$34: 3D1.A, 3L1.P2, 3U1.P4
- removed net N$35: 3C6.2, 3Q1.3, 3Q2.3, 3R4.1
- removed net N$36: 3R1.2, 3U1.P1
- removed net N$37: 3C2.1, 3R1.1
- removed net N$38: 3Q1.1, 3R3.2
- removed net N$39: 3D2.C, 3D3.C
- removed net N$40: 3C6.1, 3R5.1
- removed net N$42: 3C7.2, 3Q3.3, 3Q4.3, 3R8.1
- removed net N$43: 3Q3.1, 3R7.2
- removed net N$44: 3D4.C, 3D5.C
- removed net N$45: 3C7.1, 3R10.1
- removed net N$47: 3D6.C, 3L2.1, 4U1.P2
- removed net SCLK_POT: 3U2.2, J1.17
- removed net SOLENOID-: 3D3.A, 3J1.3, 3Q1.2, 3R5.2
- removed net SOLENOID-1: 3D5.A, 3J2.3, 3Q3.2, 3R10.2
- removed net SOLENOIDON1: 3Q2.1, 3R6.2, J1.21
- removed net SOLENOIDON2: 3Q4.1, 3R9.2, J1.23
- removed net VCC_2: 3C4.+, 3C5.+, 3D1.C, 3D2.A, 3D4.A, 3J1.1, 3J2.1, 3U2.5, 3U2.6
- net 12V: no longer 3C8.1, 4U1.P1, J3.3
- net 3.3V: no longer 3C3.1, 3U2.8
- net CSM1: now also J1.15; no longer J7.4
- net CSM2: now also J1.17; no longer J7.3
- net CSM3: now also J1.19; no longer J7.2
- net CSM4: now also J1.21; no longer J7.1
- net GND: no longer 3C1.-, 3C2.2, 3C3.2, 3C4.-, 3C5.-, 3C8.2, 3C9.-, 3D6.A, 3Q2.2, 3Q4.2, 3R2.1, 3R6.1, 3R9.1, 3U1.P3, 3U2.4, 4U1.P3, 4U1.P5, 4U1.TAB, J3.1
- net VCC_1: no longer 3C1.+, 3L1.P1, 3R3.1, 3R4.2, 3R7.1, 3R8.2, 3U1.P5

Commit message: 18/3 PCB mostly updated PCB1 layout
Parts:
- removed 1JP1, 1JP3, 1JP5: JUMPER-SMT_2_NO_SILK, SparkFun-Jumpers:SMT-JUMPER_2_NO_SILK
- removed J4, J5: (no value), SparkFun-Connectors:SCREWTERMINAL-5MM-3
- added GND: (no value), wirepad:3,17/1,1
- moved J2 170.0 mm to (-24.1, -85.1), turned to 270 degrees
- moved J1 84.1 mm to (15.2, -13.7)
- moved 1R7 39.5 mm to (-30.5, -2.54), turned to 0 degrees
- moved 1U4 27.1 mm to (-26.7, -11.4), turned to 90 degrees
- moved 1R4 18.2 mm to (-5.08, 7.62)
- moved 1R9 12.7 mm to (-24.1, -19.1)
- moved 1R8 12.7 mm to (-20.3, -19.1)
- moved R2M3 11.4 mm to (35.6, -44.5)
- moved R2M1 11.4 mm to (-34.3, 44.5)
- moved R2M2 11.4 mm to (31.8, 48.3)
- moved J6 10.2 mm to (24.1, -95.2), turned to 90 degrees
- moved R10M1 7.25 mm to (-29.2, 49.5)
- moved R10M2 7.25 mm to (36.8, 43.2)
- moved R10M3 7.25 mm to (30.5, -49.5)
- moved 1C5 5.08 mm to (-39.4, 0.00)
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Connections:
- removed net CSDIS: R9M1.1, R9M2.1, R9M3.1, R9M4.1, U1M1.P6, U1M2.P6, U1M3.P6, U1M4.P6
- new net CSDIS1: R9M1.1, U1M1.P6
- new net CSDIS2: R9M2.1, U1M2.P6
- new net CSDIS3: R9M3.1, U1M3.P6
- new net CSDIS4: R9M4.1, U1M4.P6
- net 12V: now also J2.3
- net 3.3V: now also J1.23; no longer J2.3
- net GND: now also GND.1; no longer 1JP1.1, 1JP3.1, 1JP5.1, J4.1, J5.1
- net N$67: no longer 1JP1.2
- net N$70: no longer 1JP3.2
- net N$88: no longer 1JP5.2
- net VCC_1: no longer J4.3, J5.3
Routing:
- net 3.3V: track 0.00 -> 723.7 mm, vias 0 -> 2
- net VCC_1: track 0.00 -> 545.9 mm, vias 0 -> 11
- net OUTBM4: track 0.00 -> 85.4 mm, vias 0 -> 4
- net OUTBM2: track 0.00 -> 83.7 mm, vias 0 -> 2
- net N$3: track 0.00 -> 73.3 mm, vias 0 -> 2
- net N$26: track 0.00 -> 71.8 mm, vias 0 -> 1
- net OUTAM2: track 0.00 -> 71.5 mm, vias 0 -> 2
- net OUTBM3: track 0.00 -> 70.3 mm, vias 0 -> 2
- net OUTAM4: track 0.00 -> 69.5 mm, vias 0 -> 2
- net 12V: track 0.00 -> 66.9 mm
- net OUTBM1: track 0.00 -> 64.1 mm, vias 0 -> 2
- net N$18: track 0.00 -> 62.8 mm, vias 0 -> 2
- net OUTAM1: track 0.00 -> 55.7 mm, vias 0 -> 1
- net N$9: track 0.00 -> 54.8 mm
- net N$1: track 0.00 -> 54.2 mm
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
Commit message: 19/3 Finally finished PCB everything gerber in here too bye maybe make a 3d model sometime when im free
Parts:
- moved J6 139.0 mm to (95.2, 24.1), turned to 180 degrees
- moved LED41 131.1 mm to (-92.7, 0.00), turned to 90 degrees
- moved LED47 131.1 mm to (92.7, 0.00), turned to 270 degrees
- moved GND 130.3 mm to (-90.2, -19.1), turned to 90 degrees
- moved J2 125.1 mm to (85.1, -24.1), turned to 0 degrees
- moved PT41 123.9 mm to (-87.6, 0.00), turned to 270 degrees
- moved PT47 123.9 mm to (87.6, 0.00), turned to 90 degrees
- moved D2M2 120.5 mm to (-83.8, 15.2), turned to 90 degrees
- moved D2M1 119.4 mm to (-83.8, -10.2), turned to 90 degrees
- moved D1M3 118.4 mm to (82.5, 14.0), turned to 270 degrees
- moved D1M4 117.9 mm to (82.5, -11.4), turned to 270 degrees
- moved LED40 116.7 mm to (-82.5, 0.00), turned to 90 degrees
- moved LED46 116.7 mm to (82.5, 0.00), turned to 270 degrees
- moved R12M1 115.5 mm to (-80.0, -16.5), turned to 0 degrees
- moved D1M2 115.2 mm to (-80.0, 15.2), turned to 270 degrees
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Routing:
- net GND: track 0.00 -> 1439.5 mm, vias 0 -> 29
- net S3: track 0.00 -> 343.4 mm, vias 0 -> 10
- net INAM2: track 0.00 -> 261.4 mm, vias 0 -> 8
- net N$77: track 0.00 -> 259.2 mm, vias 0 -> 8
- net N$97: track 0.00 -> 256.4 mm, vias 0 -> 6
- net GATE2: track 5.28 -> 247.9 mm, vias 0 -> 7
- net N$98: track 0.00 -> 238.5 mm, vias 0 -> 8
- net PWMM2: track 15.7 -> 239.9 mm, vias 0 -> 4
- net N$83: track 0.00 -> 220.3 mm, vias 0 -> 8
- net INBM2: track 0.00 -> 200.4 mm, vias 0 -> 6
- net N$93: track 0.00 -> 190.9 mm, vias 0 -> 6
- net N$81: track 0.00 -> 187.5 mm, vias 0 -> 8
- net N$95: track 0.00 -> 180.6 mm, vias 0 -> 6
- net N$96: track 0.00 -> 177.8 mm, vias 0 -> 4
- net INBM1: track 0.00 -> 171.9 mm, vias 0 -> 8
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Other:
- board size 190.7 x 218 mm -> 218 x 190.7 mm
- board text added: "-VE"
- board text added: "12V"
- board text added: "12V POWER PCB2"
- board text added: "3V3"
- board text added: "GND"
- board text added: "MOTOR SWITCH"
- board text added: "VCC_1"
