File: PCB/projects/PCB2k19/PCB1.sch (EAGLE design)
At the start: 253 parts, among them Q1M1 AOD482, Q1M2 AOD482, Q1M3 AOD482, Q1M4 AOD482, U1M1 VNH5019, U1M2 VNH5019, U1M3 VNH5019, U1M4 VNH5019

Commit message: 15/3 Updated the schematics, labelled of PCB2
Parts:
- added 1R12, 1R13: (no value), SparkFun-Resistors:RESISTOR0603
- added IRIN1, IRIN2, LED48, LED49: (no value), SparkFun-Connectors:CONN_03
- added J2, J3, J4, J5, J6: (no value), SparkFun-Connectors:CONN_03SCREW_LOCK
- added J7: (no value), SparkFun-Connectors:CONN_04LOCK
Connections:
- removed net N$115: J1.25
- removed net N$128: J1.26
- new net GATE1: 1R12.2, IRIN1.1, J1.25
- new net GATE2: 1R13.2, IRIN2.1, J1.26
- new net VCC_1: J4.3, J5.3, J6.1, Q1M1.S, Q1M2.S, Q1M3.S, Q1M4.S, U1M1.VBAT, U1M2.VBAT, U1M3.VBAT, U1M4.VBAT
- net 12V: now also J3.3, J6.3; no longer Q1M1.S, Q1M2.S, Q1M3.S, Q1M4.S, U1M1.VBAT, U1M2.VBAT, U1M3.VBAT, U1M4.VBAT
- net 3.3V: now also IRIN1.3, IRIN2.3, J2.3, LED48.3, LED49.3
- net 5V: now also J2.2
- net CSM1: now also J7.4
- net CSM2: now also J7.3
- net CSM3: now also J7.2
- net CSM4: now also J7.1
- net GND: now also 1R12.1, 1R13.1, J2.1, J3.1, J4.1, J5.1, LED48.1, LED49.1
Other:
- moved on the sheet: 1U1G4

Commit message: 17/3 Updated derp in Boost Circuit voltage selection, updated boards even further
Parts:
- 1R10, 1R11, 1R2, 1R5, 1R8: device rcl:R-EU_R0603 -> SparkFun-Resistors:1.5KOHM-0603-1/10W-1%
- 3C10, 3C11: device rcl:C-EUC1210 -> SparkFun-Capacitors:22UF-1210-16V-20%
- 3C12: value 10.0nF -> 10nF; device rcl:C-EUC0603 -> SparkFun-Capacitors:10NF-0603-50V-10%
- 3C6, 3C7: device rcl:C-EUC0603 -> SparkFun-Capacitors:1.5PF-0603-50V-16.667%
- 3R10, 3R5: device rcl:R-EU_R0603 -> SparkFun-Resistors:20OHM-0603-1/10W-1%
- 3R11, 3R4, 3R6, 3R8, 3R9: device rcl:R-EU_R0603 -> SparkFun-Resistors:10KOHM-0603-1/10W-1%
- 3R12: device rcl:R-EU_R0603 -> SparkFun-Resistors:5.62KOHM-0603-1/10W-1%
- 3R2: value 2.0k -> 1.69k
- 3R3, 3R7: device rcl:R-EU_R0603 -> SparkFun-Resistors:1KOHM-0603-1/10W-1%
- renumbered 1PT0 to PT0, 1PT1 to PT1, 1PT10 to PT10, 1PT11 to PT11, 1PT12 to PT12, 1PT13 to PT13, 1PT14 to PT14, 1PT15 to PT15, 1PT16 to PT16, 1PT17 to PT17, 1PT18 to PT18, 1PT19 to PT19, 1PT2 to PT2, 1PT20 to PT20, 1PT21 to PT21, 1PT22 to PT22, 1PT23 to PT23, 1PT24 to PT24, 1PT25 to PT25, 1PT26 to PT26, 1PT27 to PT27, 1PT28 to PT28, 1PT29 to PT29, 1PT3 to PT3, 1PT30 to PT30, 1PT31 to PT31, 1PT32 to PT32, 1PT33 to PT33, 1PT34 to PT34, 1PT35 to PT35, 1PT36 to PT36, 1PT37 to PT37, 1PT38 to PT38, 1PT39 to PT39, 1PT4 to PT4, 1PT40 to PT40, 1PT41 to PT41, 1PT42 to PT42, 1PT43 to PT43, 1PT44 to PT44, 1PT45 to PT45, 1PT46 to PT46, 1PT47 to PT47, 1PT5 to PT5, 1PT6 to PT6, 1PT7 to PT7, 1PT8 to PT8, 1PT9 to PT9, D12M1 to R12M1, D12M2 to R12M2, D12M3 to R12M3, D12M4 to R12M4
Connections:
- removed net N$41: 3U2.PA0, 3U2.PW0
- new net N$103: 3R2.2, 3U1.FDBK, 3U2.PB0
- net 12V: now also J6.1; no longer 3C1.+, 3L1.1, 3R3.1, 3R4.2, 3R7.1, 3R8.2, 3U1.VIN, J6.3
- net VCC_1: now also 3C1.+, 3L1.1, 3R3.1, 3R4.2, 3R7.1, 3R8.2, 3U1.VIN, J6.3; no longer J6.1
- net VCC_2: now also 3U2.PA0, 3U2.PW0; no longer 3R2.2, 3U1.FDBK, 3U2.PB0
Other:
- moved on the sheet: 3C10, 3C11

Commit message: 18/3 Moved boost circuit and solenoid circuits to PCB2 else no space
Parts:
- removed 3C1: 100uF, SparkFun-Capacitors:100UF-POLAR-25V-20%(ELEC)
- removed 3C2: 680nF, SparkFun-Capacitors:680PF-0603-50V-10%
- removed 3C3: 0.1uF, SparkFun-Capacitors:0.1UF-0603-25V-5%
- removed 3C4, 3C5: 1000uF, JH:1000UF-CAP
- removed 3C6, 3C7: 1500pF, SparkFun-Capacitors:1.5PF-0603-50V-16.667%
- removed 3C8: 22UF, SparkFun-Capacitors:22UF-1210-16V-20%
- removed 3C9: 6.8uF, rcl:CPOL-USA/3216-18R
- removed 3D1: SS510, diode:SCHOTTKY-DIODESMD
- removed 3D2, 3D4: 1N4728, diode:1N4728
- removed 3D3, 3D5: 1N5401, diode:1N5400
- removed 3D6: SS54, diode:SCHOTTKY-DIODESMD
- removed 3J1, 3J2: (no value), SparkFun-Connectors:CONN_03-SCREW-5MM
- removed 3L1: 100UH-L, JH:100UH-L
- removed 3L2: 33uH, JH:CDRH127
- removed 3Q1, 3Q3: STP75NF75, SparkFun-DiscreteSemi:MOSFET-NCH-FQP30N06L
- removed 3Q2, 3Q4: AO3400, SparkFun-DiscreteSemi:MOSFET-NCH-AO3404A
- removed 3R1: 2.94k, SparkFun-Resistors:RESISTOR0603
- removed 3R10, 3R5: 20, SparkFun-Resistors:20OHM-0603-1/10W-1%
- removed 3R2: 1.69k, SparkFun-Resistors:2.0KOHM-0603-1/10W-5%
- removed 3R3, 3R7: 1k, SparkFun-Resistors:1KOHM-0603-1/10W-1%
- removed 3R4, 3R6, 3R8, 3R9: 10k, SparkFun-Resistors:10KOHM-0603-1/10W-1%
- removed 3U1: LM2587, JH:LM2587
- removed 3U2: (no value), JH:MCP41XXX
- removed 4U1: LM2596, JH:LM2596
- removed J3: (no value), SparkFun-Connectors:CONN_03SCREW_LOCK
- removed J7: (no value), SparkFun-Connectors:CONN_04LOCK
- J2, J4, J5, J6: device SparkFun-Connectors:CONN_03SCREW_LOCK -> SparkFun-Connectors:CONN_03-SCREW-5MM
Connections:
- removed net 5V: 3C9.+, 3L2.2, 4U1.FDBK, J2.2
- removed net CS_POT: 3U2.CS, J1.15
- removed net MOSI_POT: 3U2.MOSI, J1.19
- removed net N$103: 3R2.2, 3U1.FDBK, 3U2.PB0
- removed net N$34: 3D1.A, 3L1.2, 3U1.SW
- removed net N$35: 3C6.2, 3Q1.S, 3Q2.D, 3R4.1
- removed net N$36: 3R1.2, 3U1.COMP
- removed net N$37: 3C2.1, 3R1.1
- removed net N$38: 3Q1.G, 3R3.2
- removed net N$39: 3D2.C, 3D3.C
- removed net N$40: 3C6.1, 3R5.1
- removed net N$42: 3C7.2, 3Q3.S, 3Q4.D, 3R8.1
- removed net N$43: 3Q3.G, 3R7.2
- removed net N$44: 3D4.C, 3D5.C
- removed net N$45: 3C7.1, 3R10.1
- removed net N$47: 3D6.C, 3L2.1, 4U1.OUT
- removed net SCLK_POT: 3U2.SCLK, J1.17
- removed net SOLENOID-: 3D3.A, 3J1.3, 3Q1.D, 3R5.2
- removed net SOLENOID-1: 3D5.A, 3J2.3, 3Q3.D, 3R10.2
- removed net SOLENOIDON1: 3Q2.G, 3R6.2, J1.21
- removed net SOLENOIDON2: 3Q4.G, 3R9.2, J1.23
- removed net VCC_2: 3C4.+, 3C5.+, 3D1.C, 3D2.A, 3D4.A, 3J1.1, 3J2.1, 3U2.PA0, 3U2.PW0
- net 12V: no longer 3C8.1, 4U1.VIN, J3.3
- net 3.3V: no longer 3C3.1, 3U2.VCC
- net CSM1: now also J1.15; no longer J7.4
- net CSM2: now also J1.17; no longer J7.3
- net CSM3: now also J1.19; no longer J7.2
- net CSM4: now also J1.21; no longer J7.1
- net GND: no longer 3C1.-, 3C2.2, 3C3.2, 3C4.-, 3C5.-, 3C8.2, 3C9.-, 3D6.A, 3Q2.S, 3Q4.S, 3R2.1, 3R6.1, 3R9.1, 3U1.GND, 3U2.GND, 4U1.ENA, 4U1.GND, J3.1
- net VCC_1: no longer 3C1.+, 3L1.1, 3R3.1, 3R4.2, 3R7.1, 3R8.2, 3U1.VIN
Other:
- note added: "add gnd batt connector"
- moved on the sheet: 3C10, 3C11, 3C12, 3C13, 3D7, 3L3, 3R11, 3R12, 4U2

Commit message: 18/3 PCB mostly updated PCB1 layout
Parts:
- removed 1JP1, 1JP3, 1JP5: JUMPER-SMT_2_NO_SILK, SparkFun-Jumpers:JUMPER-SMT_2_NO_SILK
- removed J4, J5: (no value), SparkFun-Connectors:CONN_03-SCREW-5MM
- added GND: (no value), wirepad:3,17/1,1
Connections:
- removed net CSDIS: R9M1.1, R9M2.1, R9M3.1, R9M4.1, U1M1.CS_DIS, U1M2.CS_DIS, U1M3.CS_DIS, U1M4.CS_DIS
- new net CSDIS1: R9M1.1, U1M1.CS_DIS
- new net CSDIS2: R9M2.1, U1M2.CS_DIS
- new net CSDIS3: R9M3.1, U1M3.CS_DIS
- new net CSDIS4: R9M4.1, U1M4.CS_DIS
- net 12V: now also J2.3
- net 3.3V: now also J1.23; no longer J2.3
- net GND: now also GND.P; no longer 1JP1.1, 1JP3.1, 1JP5.1, J4.1, J5.1
- net N$67: no longer 1JP1.2
- net N$70: no longer 1JP3.2
- net N$88: no longer 1JP5.2
- net VCC_1: no longer J4.3, J5.3
Other:
- note removed: "add gnd batt connector"
