File: PCB/projects/PCB2k19/PCB2.brd (EAGLE design)
At the start: 192.8 x 160 mm, 24 parts

Commit message: 15/3 Updated the schematics, labelled of PCB2
Parts:
- added J19: (no value), SparkFun-Connectors:SCREWTERMINAL-3.5MM-3_LOCK.007S
- added J20, J21: (no value), SparkFun-Connectors:1X30
- added J22, J23, J24, J25: (no value), SparkFun-Connectors:1X20
- added J26: (no value), SparkFun-Connectors:1X02_LOCK
- added J27: (no value), SparkFun-Connectors:1X04_LOCK
- moved J12 153.3 mm to (33.0, -68.6), turned to 180 degrees
- moved J18 144.4 mm to (-55.9, 43.2), turned to 180 degrees
- moved S1 141.4 mm to (16.5, -68.6), turned to 270 degrees
- moved U$3 133.0 mm to (-48.3, 45.7), turned to 0 degrees
- moved J2 132.3 mm to (3.81, 66.0), turned to 180 degrees
- moved J4 132.3 mm to (-3.81, -66.0), turned to 0 degrees
- moved J1 129.4 mm to (-15.2, 73.7), turned to 180 degrees
- moved J3 116.9 mm to (1.27, 58.4), turned to 180 degrees
- moved J5 116.9 mm to (-1.27, -58.4), turned to 0 degrees
- moved J17 111.9 mm to (-43.2, 35.6), turned to 180 degrees
- moved R2 110.3 mm to (-26.7, 48.3), turned to 180 degrees
- moved J6 107.0 mm to (53.3, -3.81), turned to 90 degrees
- moved J8 107.0 mm to (-53.3, 3.81), turned to 270 degrees
- moved U$2 106.1 mm to (35.6, 39.4), turned to 270 degrees
- moved R1 105.9 mm to (-26.7, 45.7), turned to 180 degrees
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Connections:
- new net P43: J27.4, U$1.43
- new net P44: J27.3, U$1.44
- new net P49: J27.2, U$1.49/A23
- new net P50: J27.1, U$1.50/A24
- net 3.3V: now also J19.3
- net 5V: now also J19.2
- net GND: now also J19.1, J26.1
- net IN1: now also U$1.45
- net IN2: now also U$1.48
- net N$1: now also J26.2
Routing:
- net 5V: track 0.00 -> 16.0 mm
- net PWMESC2: track 0.00 -> 8.03 mm
- net PWMESC1: track 0.00 -> 7.50 mm
Other:
- outline, holes or cut-outs redrawn
- board text added: "(NC)"
- board text added: "3V3"
- board text added: "3v3"
- board text added: "5V"
- board text added: "74HCT08 AND GATE"
- board text added: "ADXL345"
- board text added: "AT Mode"
- board text added: "ATX"
- board text added: "BNO055 Compass"
- board text added: "BOOT"
- board text added: "CS"
- board text added: "DATA"
- board text added: "Data Mode"
- board text added: "ESC"
- board text added: "GND"
- board text added: "GPIO"
- board text added: "HC-05 Bluetooth"
- board text added: "I2C"
- board text added: "IN1"
- board text added: "IN2"
- board text added: "INT"
- board text added: "KEY"
- board text added: "LRX"
- board text added: "MISO"
- board text added: "MOSI"
- board text added: "NEOPIXEL RING"
- board text added: "OFF"
- board text added: "ON"
- board text added: "P43"
- board text added: "P44"
- board text added: "P49"
- board text added: "P50"
- board text added: "RASPI POWER"
- board text added: "RASPI SERIAL"
- board text added: "RASPI USB"
- board text added: "RES"
- board text added: "RX"
- board text added: "SCL"
- board text added: "SCLK"
- board text added: "SDA"
- board text added: "STATE"
- board text added: "TX"
- board text added: "VIN"
- board text added: "VL53L0X TOF"
- board text added: "VS"
- board text added: "XSHUT"

Commit message: 17/3 Updated derp in Boost Circuit voltage selection, updated boards even further
Parts:
- moved J20 168.9 mm to (61.0, 58.4), turned to 270 degrees
- moved J21 165.2 mm to (58.4, 58.4), turned to 270 degrees
- moved J22 161.7 mm to (55.9, 58.4), turned to 270 degrees
- moved J23 158.2 mm to (53.3, 58.4), turned to 270 degrees
- moved J24 154.8 mm to (50.8, 58.4), turned to 270 degrees
- moved J12 152.2 mm to (-33.0, 68.6), turned to 0 degrees
- moved J25 151.6 mm to (48.3, 58.4), turned to 270 degrees
- moved J1 150.4 mm to (15.2, -73.7), turned to 0 degrees
- moved J18 141.2 mm to (55.9, -43.2), turned to 0 degrees
- moved S1 141.1 mm to (-16.5, 68.6), turned to 90 degrees
- moved U$3 133.0 mm to (48.3, -45.7), turned to 180 degrees
- moved J2 132.3 mm to (-3.81, -66.0), turned to 0 degrees
- moved J4 132.3 mm to (3.81, 66.0), turned to 180 degrees
- moved J3 116.9 mm to (-1.27, -58.4), turned to 0 degrees
- moved J5 116.9 mm to (1.27, 58.4), turned to 180 degrees
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Other:
- outline, holes or cut-outs redrawn

Commit message: 18/3 Moved boost circuit and solenoid circuits to PCB2 else no space
Parts:
- removed J27: (no value), SparkFun-Connectors:1X04_LOCK
- added 3C1: 100uF, SparkFun-Capacitors:PANASONIC_D
- added 3C2: 680nF, SparkFun-Capacitors:0603
- added 3C3: 0.1uF, SparkFun-Capacitors:0603
- added 3C4, 3C5: 1000uF, JH:1000UF-CAP
- added 3C6, 3C7: 1500pF, SparkFun-Capacitors:0603
- added 3C8: 22UF, SparkFun-Capacitors:1210
- added 3C9: 6.8uF, rcl:A/3216-18R
- added 3D1: SS510, diode:SMB
- added 3D2, 3D4: 1N4728, diode:DO41Z10
- added 3D3, 3D5: 1N5401, diode:DO201-15
- added 3D6: SS54, diode:SMB
- added 3J1, 3J2: (no value), SparkFun-Connectors:SCREWTERMINAL-5MM-3
- added 3L1: 100UH-L, JH:100UH-L
- added 3L2: 33uH, JH:127
- added 3Q1, 3Q3: STP75NF75, SparkFun-DiscreteSemi:TO220V
- added 3Q2, 3Q4: AO3400, SparkFun-DiscreteSemi:SOT23-3
- added 3R1: 2.94k, SparkFun-Resistors:0603
- added 3R10, 3R5: 20, SparkFun-Resistors:0603
- added 3R2: 1.69k, SparkFun-Resistors:0603
- added 3R3, 3R7: 1k, SparkFun-Resistors:0603
- added 3R4, 3R6, 3R8, 3R9: 10k, SparkFun-Resistors:0603
- added 3U1: LM2587, JH:TO-263
- added 3U2: (no value), JH:SOIC-8
- added 4U1: LM2596, JH:TO-263
- J19: device SparkFun-Connectors:SCREWTERMINAL-3.5MM-3_LOCK.007S -> SparkFun-Connectors:SCREWTERMINAL-5MM-3
- moved J21 93.4 mm to (149.9, 39.4)
- moved J24 93.4 mm to (142.2, 39.4)
- moved J20 93.4 mm to (152.4, 39.4)
- moved J22 93.4 mm to (147.3, 39.4)
- moved J23 93.4 mm to (144.8, 39.4)
- moved J25 93.4 mm to (139.7, 39.4)
- moved J19 8.89 mm to (-11.4, -48.3), turned to 180 degrees
Connections:
- removed net P43: J27.4, U$1.43
- removed net P44: J27.3, U$1.44
- removed net P49: J27.2, U$1.49/A23
- removed net P50: J27.1, U$1.50/A24
- new net 12V: 3C1.+, 3C8.1, 3L1.P1, 3U1.P5, 4U1.P1
- new net CSM1: J1.15, U$1.43
- new net CSM2: J1.17, U$1.44
- new net CSM3: J1.19, U$1.45
- new net CSM4: J1.21, U$1.46
- new net MOSI_POT: 3U2.3
- new net N$103: 3R2.2, 3U1.P2, 3U2.7
- new net N$34: 3D1.A, 3L1.P2, 3U1.P4
- new net N$35: 3C6.2, 3Q1.3, 3Q2.3, 3R4.1
- new net N$36: 3R1.2, 3U1.P1
- new net N$37: 3C2.1, 3R1.1
- new net N$38: 3Q1.1, 3R3.2
- new net N$39: 3D2.C, 3D3.C
- new net N$40: 3C6.1, 3R5.1
- new net N$42: 3C7.2, 3Q3.3, 3Q4.3, 3R8.1
- new net N$43: 3Q3.1, 3R7.2
- new net N$44: 3D4.C, 3D5.C
- new net N$45: 3C7.1, 3R10.1
- new net N$47: 3D6.C, 3L2.1, 4U1.P2
- new net SCLK_POT: 3U2.2
- new net SOLENOID-: 3D3.A, 3J1.3, 3Q1.2, 3R5.2
- new net SOLENOID-1: 3D5.A, 3J2.3, 3Q3.2, 3R10.2
- new net VCC_1: 3R3.1, 3R4.2, 3R7.1, 3R8.2
- new net VCC_2: 3C4.+, 3C5.+, 3D1.C, 3D2.A, 3D4.A, 3J1.1, 3J2.1, 3U2.5, 3U2.6
- net 3.3V: now also 3C3.1, 3U2.8
- net 5V: now also 3C9.+, 3L2.2, 4U1.P4; no longer J19.2
- net CS_POT: now also 3U2.1; no longer J1.15
- net GND: now also 3C1.-, 3C2.2, 3C3.2, 3C4.-, 3C5.-, 3C8.2, 3C9.-, 3D6.A, 3Q2.2, 3Q4.2, 3R2.1, 3R6.1, 3R9.1, 3U1.P3, 3U2.4, 4U1.P3, 4U1.P5, 4U1.TAB
- net IN1: now also U$1.50/A24; no longer U$1.45
- net IN2: now also U$1.49/A23; no longer U$1.48
- net MOSI: no longer J1.19
- net SCLK: no longer J1.17
- net SOLENOIDON1: now also 3Q2.1, 3R6.2; no longer J1.21
- net SOLENOIDON2: now also 3Q4.1, 3R9.2; no longer J1.23
- net XSHUT3: now also U$1.48; no longer U$1.46
Other:
- board text removed: "P43"
- board text removed: "P44"
- board text removed: "P49"
- board text removed: "P50"

Commit message: 18/3 PCB mostly updated PCB1 layout
Parts:
- removed 3C5: 1000uF, JH:1000UF-CAP
- removed 3J1: (no value), SparkFun-Connectors:SCREWTERMINAL-5MM-3
- removed J11: (no value), SparkFun-Connectors:1X05_LOCK
- removed J24, J25: (no value), SparkFun-Connectors:1X20
- added C13, C22: 0.1uF, SparkFun-Capacitors:0603
- added C23: 10uf, rcl:R/2012-12R
- added U3: ADXL345, SparkFun-Sensors:LGA-14
- 3C4: value 1000uF -> 1500uF
- J10: device SparkFun-Connectors:1X05_LOCK -> SparkFun-Connectors:SCREWTERMINAL-5MM-3
- moved 3J2 164.6 mm to (27.9, 2.54)
- moved 3R7 149.4 mm to (7.62, -25.4), flipped to the bottom, turned to 270 degrees
- moved 3Q3 148.2 mm to (12.7, -34.3), turned to 270 degrees
- moved 3C3 146.3 mm to (-27.9, 17.8), turned to 270 degrees
- moved 3C2 145.5 mm to (-17.8, 19.1), turned to 180 degrees
- moved 3R8 145.1 mm to (3.81, -25.4), flipped to the bottom, turned to 180 degrees
- moved 3R1 144.9 mm to (-14.0, 19.1), turned to 0 degrees
- moved 3U2 144.3 mm to (-22.9, 17.8), turned to 90 degrees
- moved 3R6 143.8 mm to (-6.35, -25.4), flipped to the bottom
- moved 3R3 141.7 mm to (-10.2, -33.0), flipped to the bottom, turned to 90 degrees
- moved 3R4 141.7 mm to (-6.35, -33.0), flipped to the bottom
- moved 3R5 140.6 mm to (-10.2, -29.2), flipped to the bottom, turned to 270 degrees
- moved 3U1 139.9 mm to (1.27, 19.1), turned to 180 degrees
- moved 3R10 139.9 mm to (7.62, -29.2), flipped to the bottom, turned to 90 degrees
- moved 3D4 137.9 mm to (-6.35, -16.5), turned to 180 degrees
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Connections:
- removed net IN1: J11.1, U$1.50/A24
- removed net IN2: J11.2, U$1.49/A23
- removed net N$2: J10.2
- removed net N$5: J10.5
- removed net VCC_1: 3R3.1, 3R4.2, 3R7.1, 3R8.2
- new net INT1: U$1.50/A24, U3.8
- new net INT2: U$1.49/A23, U3.9
- new net N$7: 3C4.+, 3D1.C, 3U2.5, 3U2.6
- net 12V: now also 3R3.1, 3R4.2, 3R7.1, 3R8.2, J10.3, J19.3
- net 3.3V: now also C13.1, C22.1, C23.+, J1.23, U3.1, U3.6; no longer J10.4, J19.3
- net CS_ADXL: now also U3.7; no longer J10.1
- net GND: now also C13.2, C22.2, C23.-, J10.1, U3.2, U3.4, U3.5; no longer 3C5.-, J10.3
- net MISO: now also U3.12; no longer J11.3
- net MOSI: now also U3.13; no longer J11.4
- net SCLK: now also U3.14; no longer J11.5
- net SOLENOID-: now also 3J2.2; no longer 3J1.3
- net VCC_2: no longer 3C4.+, 3C5.+, 3D1.C, 3J1.1, 3U2.5, 3U2.6
Routing:
- net N$103: track 0.00 -> 20.2 mm
- net 5V: track 16.0 -> 33.9 mm
- net N$47: track 0.00 -> 16.3 mm
- net 12V: track 0.00 -> 8.98 mm
- net N$36: track 0.00 -> 5.30 mm
- net 3.3V: track 0.00 -> 3.84 mm
- net N$37: track 0.00 -> 2.11 mm
- net PWMESC2: track 8.03 -> 6.01 mm
- net PWMESC1: track 7.50 -> 5.49 mm
- net N$7: track 0.00 -> 1.27 mm
Other:
- board text added: "12v"
- board text removed: "3v3"
- board text removed: "ADXL345"
- board text removed: "CS"
- board text removed: "IN1"
- board text removed: "IN2"
- board text removed: "MISO"
- board text removed: "MOSI"
- board text removed: "SCLK"
- board text removed: "VIN"
- board text removed: "VS"

Commit message: 19/3 Finally finished PCB everything gerber in here too bye maybe make a 3d model sometime when im free
Parts:
- moved 3D1 33.5 mm to (-14.0, 7.62), turned to 0 degrees
- moved J14 11.4 mm to (5.08, -44.5), flipped to the top, turned to 270 degrees
- moved 3L1 2.84 mm to (-27.9, -8.89), turned to 0 degrees
- moved 3R2 2.54 mm to (-16.5, 15.2)
- moved J16 2.54 mm to (10.2, -44.5)
- flipped J15 to the top
Connections:
- removed net N$7: 3C4.+, 3D1.C, 3U2.5, 3U2.6
- net VCC_2: now also 3C4.+, 3D1.C, 3U2.5, 3U2.6
Routing:
- net GND: track 0.00 -> 690.9 mm, vias 0 -> 8
- net 3.3V: track 3.84 -> 682.8 mm, vias 0 -> 10
- net SDA: track 0.00 -> 402.0 mm, vias 0 -> 7
- net 5V: track 33.9 -> 419.5 mm, vias 0 -> 4
- net SCL: track 0.00 -> 341.1 mm, vias 0 -> 7
- net LSOUT1: track 0.00 -> 327.0 mm, vias 0 -> 5
- net N$6: track 0.00 -> 260.1 mm, vias 0 -> 7
- net NEOPIXEL: track 0.00 -> 243.8 mm, vias 0 -> 5
- net CSM3: track 0.00 -> 231.4 mm, vias 0 -> 4
- net LSOUT2: track 0.00 -> 229.0 mm, vias 0 -> 3
- net 12V: track 8.98 -> 238.0 mm, vias 0 -> 5
- net RX: track 0.00 -> 222.7 mm, vias 0 -> 4
- net PWMESC2: track 6.01 -> 222.9 mm, vias 0 -> 5
- net TX: track 0.00 -> 197.4 mm, vias 0 -> 4
- net LSOUT3: track 0.00 -> 195.9 mm, vias 0 -> 3
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Other:
- board text added: "1500uF"
- board text added: "60v"
- board text added: "ESC Power"
- board text added: "INDUCTOR"
- board text added: "LM2587"
- board text added: "LM2596"
- board text added: "SOLE-1"
- board text added: "SOLE-2"
- board text removed: "(NC)"
