File: PCB/projects/PCB2k19/PCB2.sch (EAGLE design)
At the start: 24 parts

Commit message: 15/3 Updated the schematics, labelled of PCB2
Parts:
- added J19: (no value), SparkFun-Connectors:CONN_03SCREW_LOCK
- added J20, J21: (no value), SparkFun-Connectors:CONN_30
- added J22, J23, J24, J25: (no value), SparkFun-Connectors:CONN_20
- added J26: (no value), SparkFun-Connectors:CONN_02LOCK
- added J27: (no value), SparkFun-Connectors:CONN_04LOCK
Connections:
- new net P43: J27.4, U$1.43
- new net P44: J27.3, U$1.44
- new net P49: J27.2, U$1.49/A23
- new net P50: J27.1, U$1.50/A24
- net 3.3V: now also J19.3
- net 5V: now also J19.2
- net GND: now also J19.1, J26.1
- net IN1: now also U$1.45
- net IN2: now also U$1.48
- net N$1: now also J26.2
Other:
- note added: "maple mini add breakout pin"

Commit message: 18/3 Moved boost circuit and solenoid circuits to PCB2 else no space
Parts:
- removed J27: (no value), SparkFun-Connectors:CONN_04LOCK
- added 3C1: 100uF, SparkFun-Capacitors:100UF-POLAR-25V-20%(ELEC)
- added 3C2: 680nF, SparkFun-Capacitors:680PF-0603-50V-10%
- added 3C3: 0.1uF, SparkFun-Capacitors:0.1UF-0603-25V-5%
- added 3C4, 3C5: 1000uF, JH:1000UF-CAP
- added 3C6, 3C7: 1500pF, SparkFun-Capacitors:1.5PF-0603-50V-16.667%
- added 3C8: 22UF, SparkFun-Capacitors:22UF-1210-16V-20%
- added 3C9: 6.8uF, rcl:CPOL-USA/3216-18R
- added 3D1: SS510, diode:SCHOTTKY-DIODESMD
- added 3D2, 3D4: 1N4728, diode:1N4728
- added 3D3, 3D5: 1N5401, diode:1N5400
- added 3D6: SS54, diode:SCHOTTKY-DIODESMD
- added 3J1, 3J2: (no value), SparkFun-Connectors:CONN_03-SCREW-5MM
- added 3L1: 100UH-L, JH:100UH-L
- added 3L2: 33uH, JH:CDRH127
- added 3Q1, 3Q3: STP75NF75, SparkFun-DiscreteSemi:MOSFET-NCH-FQP30N06L
- added 3Q2, 3Q4: AO3400, SparkFun-DiscreteSemi:MOSFET-NCH-AO3404A
- added 3R1: 2.94k, SparkFun-Resistors:RESISTOR0603
- added 3R10, 3R5: 20, SparkFun-Resistors:20OHM-0603-1/10W-1%
- added 3R2: 1.69k, SparkFun-Resistors:2.0KOHM-0603-1/10W-5%
- added 3R3, 3R7: 1k, SparkFun-Resistors:1KOHM-0603-1/10W-1%
- added 3R4, 3R6, 3R8, 3R9: 10k, SparkFun-Resistors:10KOHM-0603-1/10W-1%
- added 3U1: LM2587, JH:LM2587
- added 3U2: (no value), JH:MCP41XXX
- added 4U1: LM2596, JH:LM2596
- J19: device SparkFun-Connectors:CONN_03SCREW_LOCK -> SparkFun-Connectors:CONN_03-SCREW-5MM
Connections:
- removed net P43: J27.4, U$1.43
- removed net P44: J27.3, U$1.44
- removed net P49: J27.2, U$1.49/A23
- removed net P50: J27.1, U$1.50/A24
- new net 12V: 3C1.+, 3C8.1, 3L1.1, 3U1.VIN, 4U1.VIN
- new net CSM1: J1.15, U$1.43
- new net CSM2: J1.17, U$1.44
- new net CSM3: J1.19, U$1.45
- new net CSM4: J1.21, U$1.46
- new net MOSI_POT: 3U2.MOSI
- new net N$103: 3R2.2, 3U1.FDBK, 3U2.PB0
- new net N$34: 3D1.A, 3L1.2, 3U1.SW
- new net N$35: 3C6.2, 3Q1.S, 3Q2.D, 3R4.1
- new net N$36: 3R1.2, 3U1.COMP
- new net N$37: 3C2.1, 3R1.1
- new net N$38: 3Q1.G, 3R3.2
- new net N$39: 3D2.C, 3D3.C
- new net N$40: 3C6.1, 3R5.1
- new net N$42: 3C7.2, 3Q3.S, 3Q4.D, 3R8.1
- new net N$43: 3Q3.G, 3R7.2
- new net N$44: 3D4.C, 3D5.C
- new net N$45: 3C7.1, 3R10.1
- new net N$47: 3D6.C, 3L2.1, 4U1.OUT
- new net SCLK_POT: 3U2.SCLK
- new net SOLENOID-: 3D3.A, 3J1.3, 3Q1.D, 3R5.2
- new net SOLENOID-1: 3D5.A, 3J2.3, 3Q3.D, 3R10.2
- new net VCC_1: 3R3.1, 3R4.2, 3R7.1, 3R8.2
- new net VCC_2: 3C4.+, 3C5.+, 3D1.C, 3D2.A, 3D4.A, 3J1.1, 3J2.1, 3U2.PA0, 3U2.PW0
- net 3.3V: now also 3C3.1, 3U2.VCC
- net 5V: now also 3C9.+, 3L2.2, 4U1.FDBK; no longer J19.2
- net CS_POT: now also 3U2.CS; no longer J1.15
- net GND: now also 3C1.-, 3C2.2, 3C3.2, 3C4.-, 3C5.-, 3C8.2, 3C9.-, 3D6.A, 3Q2.S, 3Q4.S, 3R2.1, 3R6.1, 3R9.1, 3U1.GND, 3U2.GND, 4U1.ENA, 4U1.GND
- net IN1: now also U$1.50/A24; no longer U$1.45
- net IN2: now also U$1.49/A23; no longer U$1.48
- net MOSI: no longer J1.19
- net SCLK: no longer J1.17
- net SOLENOIDON1: now also 3Q2.G, 3R6.2; no longer J1.21
- net SOLENOIDON2: now also 3Q4.G, 3R9.2; no longer J1.23
- net XSHUT3: now also U$1.48; no longer U$1.46
Other:
- note added: "Bluetooth"
- note added: "maple mini add breakout pin add 12v in"
- note removed: "maple mini add breakout pin"

Commit message: 18/3 PCB mostly updated PCB1 layout
Parts:
- removed 3C5: 1000uF, JH:1000UF-CAP
- removed 3J1: (no value), SparkFun-Connectors:CONN_03-SCREW-5MM
- removed J11: (no value), SparkFun-Connectors:CONN_05LOCK
- removed J24, J25: (no value), SparkFun-Connectors:CONN_20
- added C13, C22: 0.1uF, SparkFun-Capacitors:0.1UF-0603-100V-10%
- added C23: 10uf, rcl:CPOL-USR/2012-12R
- added U3: ADXL345, SparkFun-Sensors:ADXL345
- 3C4: value 1000uF -> 1500uF
- J10: device SparkFun-Connectors:CONN_05LOCK -> SparkFun-Connectors:CONN_03-SCREW-5MM
Connections:
- removed net IN1: J11.1, U$1.50/A24
- removed net IN2: J11.2, U$1.49/A23
- removed net N$2: J10.2
- removed net N$5: J10.5
- removed net VCC_1: 3R3.1, 3R4.2, 3R7.1, 3R8.2
- new net INT1: U$1.50/A24, U3.INT1
- new net INT2: U$1.49/A23, U3.INT2
- new net N$7: 3C4.+, 3D1.C, 3U2.PA0, 3U2.PW0
- net 12V: now also 3R3.1, 3R4.2, 3R7.1, 3R8.2, J10.3, J19.3
- net 3.3V: now also C13.1, C22.1, C23.+, J1.23, U3.VDD, U3.VS; no longer J10.4, J19.3
- net CS_ADXL: now also U3.CS; no longer J10.1
- net GND: now also C13.2, C22.2, C23.-, J10.1, U3.GND@2, U3.GND@4, U3.GND@5; no longer 3C5.-, J10.3
- net MISO: now also U3.SDO; no longer J11.3
- net MOSI: now also U3.SDA; no longer J11.4
- net SCLK: now also U3.SCL; no longer J11.5
- net SOLENOID-: now also 3J2.2; no longer 3J1.3
- net VCC_2: no longer 3C4.+, 3C5.+, 3D1.C, 3J1.1, 3U2.PA0, 3U2.PW0
Other:
- note removed: "maple mini add breakout pin add 12v in"
- moved on the sheet: J19

Commit message: 19/3 Finally finished PCB everything gerber in here too bye maybe make a 3d model sometime when im free
Connections:
- removed net N$7: 3C4.+, 3D1.C, 3U2.PA0, 3U2.PW0
- net VCC_2: now also 3C4.+, 3D1.C, 3U2.PA0, 3U2.PW0
Changed lines of the file:
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@@
 <drawing>
 <settings>
-<setting alwaysvectorfont="yes"/>
+<setting alwaysvectorfont="no"/>
 <setting verticaltext="up"/>
 </settings>
@@
 <wire x1="231.14" y1="165.1" x2="231.14" y2="160.02" width="0.1524" layer="91"/>
 </segment>
+<segment>
+<pinref part="3D1" gate="G$1" pin="C"/>
+<wire x1="71.12" y1="157.48" x2="91.44" y2="157.48" width="0.1524" layer="91"/>
+<pinref part="3U2" gate="G$1" pin="PA0"/>
+<pinref part="3U2" gate="G$1" pin="PW0"/>
+<wire x1="91.44" y1="149.86" x2="93.98" y2="149.86" width="0.1524" layer="91"/>
+<wire x1="91.44" y1="149.86" x2="91.44" y2="157.48" width="0.1524" layer="91"/>
+<junction x="91.44" y="149.86"/>
+<wire x1="91.44" y1="157.48" x2="101.6" y2="157.48" width="0.1524" layer="91"/>
+<junction x="91.44" y="157.48"/>
+<pinref part="3C4" gate="G$1" pin="+"/>
+<wire x1="101.6" y1="157.48" x2="101.6" y2="147.32" width="0.1524" layer="91"/>
+<pinref part="SUPPLY21" gate="G$1" pin="VCC_2"/>
+<wire x1="101.6" y1="160.02" x2="101.6" y2="157.48" width="0.1524" layer="91"/>
+<junction x="101.6" y="157.48"/>
+</segment>
 </net>
 <net name="SOLENOIDON1" class="0">
@@
 </segment>
 </net>
-<net name="N$7" class="0">
-<segment>
-<pinref part="3D1" gate="G$1" pin="C"/>
-<pinref part="3C4" gate="G$1" pin="+"/>
-<wire x1="71.12" y1="157.48" x2="91.44" y2="157.48" width="0.1524" layer="91"/>
-<wire x1="91.44" y1="157.48" x2="101.6" y2="157.48" width="0.1524" layer="91"/>
-<wire x1="101.6" y1="157.48" x2="101.6" y2="147.32" width="0.1524" layer="91"/>
-<pinref part="3U2" gate="G$1" pin="PA0"/>
-<pinref part="3U2" gate="G$1" pin="PW0"/>
-<wire x1="91.44" y1="149.86" x2="93.98" y2="149.86" width="0.1524" layer="91"/>
-<wire x1="91.44" y1="149.86" x2="91.44" y2="157.48" width="0.1524" layer="91"/>
-<junction x="91.44" y="149.86"/>
-<junction x="91.44" y="157.48"/>
-<pinref part="SUPPLY21" gate="G$1" pin="VCC_2"/>
-<wire x1="101.6" y1="157.48" x2="101.6" y2="160.02" width="0.1524" layer="91"/>
-<junction x="101.6" y="157.48"/>
-</segment>
-</net>
